File: USB3-2.kicad_sch (KiCad schematic)
At the start: 45 parts, among them J4 632723300011, Q3 PJE138K, U12 AP22615A_TSOT26, U14 TPD4E05U06QDQARQ1, U15 TPD4E05U06QDQARQ1, U16 TPD4E05U06QDQARQ1, U2 HD3SS3220RNH

Commit message: v2.0 Schematic updates
Other:
- company: Argus-1 Cubesat -> Carnegie Mellon University
- title: Jetson Carrier Board -> Argus Carrierboard
Changed lines of the file:
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@@
 	(paper "A3")
 	(title_block
-		(title "Jetson Carrier Board")
-		(date "2024-07-05")
-		(rev "v1")
-		(company "Argus-1 Cubesat")
+		(title "Argus Carrierboard")
+		(date "2025-03-10")
+		(rev "v2.0")
+		(company "Carnegie Mellon University")
 		(comment 1 "www.antmicro.com")
 		(comment 2 "N. Khera")
@@
 	(label "USBSS0_TX_C_N"
 		(at 153.035 167.64 180)
-		(fields_autoplaced yes)
 		(effects
 			(font
@@
 	(label "USBC0_ADDR"
 		(at 138.43 175.26 0)
-		(fields_autoplaced yes)
 		(effects
 			(font
@@
 	(label "USBC0_DIR"
 		(at 182.88 124.46 0)
-		(fields_autoplaced yes)
 		(effects
 			(font
@@
 	(label "USBC0_CONN_TX1_P"
 		(at 224.155 170.18 0)
-		(fields_autoplaced yes)
 		(effects
 			(font
@@
 	(label "USBC0_RX2_N"
 		(at 183.515 175.26 0)
-		(fields_autoplaced yes)
 		(effects
 			(font
@@
 	(label "USBC0_FAULT_N"
 		(at 182.88 129.54 0)
-		(fields_autoplaced yes)
 		(effects
 			(font
@@
 	(label "USBC0_PORT"
 		(at 137.795 142.24 0)
-		(fields_autoplaced yes)
 		(effects
 			(font
@@
 	(label "USBC0_ISC_SCL"
 		(at 138.43 180.34 0)
-		(fields_autoplaced yes)
 		(effects
 			(font
@@
 	(label "USBC0_CONN_TX2_N"
 		(at 224.155 182.88 0)
-		(fields_autoplaced yes)
 		(effects
 			(font
@@
 	(label "USBC0_ID"
 		(at 182.88 127 0)
-		(fields_autoplaced yes)
 		(effects
 			(font
@@
 	(label "USBC0_CC1"
 		(at 224.155 139.7 0)
-		(fields_autoplaced yes)
 		(effects
 			(font
@@
 	(label "USBC0_I2C_SDA"
 		(at 111.76 196.85 0)
-		(fields_autoplaced yes)
 		(effects
 			(font
@@
 	(label "USBC0_I_MODE"
 		(at 137.795 139.7 0)
-		(fields_autoplaced yes)
 		(effects
 			(font
@@
 	(label "USBC0_VBUS_DET"
 		(at 182.88 134.62 0)
-		(fields_autoplaced yes)
 		(effects
 			(font
@@
 	(label "USBC0_RX1_P"
 		(at 183.515 162.56 0)
-		(fields_autoplaced yes)
 		(effects
 			(font
@@
 	(label "USBC0_CC2"
 		(at 224.155 142.24 0)
-		(fields_autoplaced yes)
 		(effects
 			(font
@@
 	(label "USBC0_VBUS"
 		(at 255.27 91.44 0)
-		(fields_autoplaced yes)
 		(effects
 			(font
@@
 	(label "USBC0_CONN_TX2_P"
 		(at 224.155 185.42 0)
-		(fields_autoplaced yes)
 		(effects
 			(font
@@
 	(label "USBC0_ISC_SCL"
 		(at 111.76 199.39 0)
-		(fields_autoplaced yes)
 		(effects
 			(font
@@
 	(label "~{USBC0_EN_MUX}"
 		(at 137.795 144.78 0)
-		(fields_autoplaced yes)
 		(effects
 			(font
@@
 	(label "USBC0_INT"
 		(at 138.43 182.88 0)
-		(fields_autoplaced yes)
 		(effects
 			(font
@@
 	(label "USBC0_TX2_N"
 		(at 183.515 182.88 0)
-		(fields_autoplaced yes)
 		(effects
 			(font
@@
 	(label "USBC0_TX1_P"
 		(at 183.515 170.18 0)
-		(fields_autoplaced yes)
 		(effects
 			(font
@@
 	(label "USBC0_FLG"
 		(at 229.87 93.98 0)
-		(fields_autoplaced yes)
 		(effects
 			(font
@@
 	(label "USBC0_RX1_N"
 		(at 183.515 160.02 0)
-		(fields_autoplaced yes)
 		(effects
 			(font
@@
 	(label "USBC0_TX1_N"
 		(at 183.515 167.64 0)
-		(fields_autoplaced yes)
 		(effects
 			(font
@@
 	(label "USBSS0_TX_C_P"
 		(at 153.035 170.18 180)
-		(fields_autoplaced yes)
 		(effects
 			(font
@@
 	(label "USBC0_I2C_SDA"
 		(at 138.43 177.8 0)
-		(fields_autoplaced yes)
 		(effects
 			(font
@@
 	(label "~{USBC0_EN_CC}"
 		(at 137.795 147.32 0)
-		(fields_autoplaced yes)
 		(effects
 			(font
@@
 	(label "USBSS0_RX_C_P"
 		(at 153.035 162.56 180)
-		(fields_autoplaced yes)
 		(effects
 			(font
@@
 	(label "USBC0_RX2_P"
 		(at 183.515 177.8 0)
-		(fields_autoplaced yes)
 		(effects
 			(font
@@
 	(label "USBC0_ISET"
 		(at 255.27 93.98 0)
-		(fields_autoplaced yes)
 		(effects
 			(font
@@
 	(label "USBC0_CONN_TX1_N"
 		(at 224.155 167.64 0)
-		(fields_autoplaced yes)
 		(effects
 			(font
@@
 	(label "USBC0_TX2_P"
 		(at 183.515 185.42 0)
-		(fields_autoplaced yes)
 		(effects
 			(font
@@
 	(label "USBSS0_RX_C_N"
 		(at 153.035 160.02 180)
-		(fields_autoplaced yes)
-		(effects
-			(font
+		(effects
+			(font
