File: USB3-2.kicad_sch (KiCad schematic)
At the start: 45 parts, among them J4 632723300011, Q3 PJE138K, U12 AP22615A_TSOT26, U14 TPD4E05U06QDQARQ1, U15 TPD4E05U06QDQARQ1, U16 TPD4E05U06QDQARQ1, U2 HD3SS3220RNH

Commit message: Clean up silk, BOM
Parts:
- C10, C57, C60, C61, C62, C63, C8, C9: LCSC (none) -> C14663
- C11: LCSC (none) -> C16772
- C7: LCSC (none) -> C84419
- D7, D8: LCSC (none) -> C87910
- J4: LCSC (none) -> C3197928
- Q3: LCSC (none) -> C391643
- R104, R22: LCSC (none) -> C25804
- R106: LCSC (none) -> C108943
- R14, R15, R16, R20: LCSC (none) -> C17168
- R17, R18: LCSC (none) -> C25792
- R21: LCSC (none) -> C21189
- R27, R42, R43: LCSC (none) -> C23162
- R28, R29: LCSC (none) -> C227752
- R30, R45: LCSC (none) -> C23186
- R32, R33: LCSC (none) -> C21190
- R41, R83: LCSC (none) -> C4190
- R44: LCSC (none) -> C22935
- R52: LCSC (none) -> C4125
- U12: LCSC (none) -> C2687851
- U14, U15: LCSC (none) -> C81353
- U16: LCSC (none) -> C2674581
- U2: LCSC (none) -> C892821
