File: hdmi.kicad_sch (KiCad schematic)
At the start: 41 parts, among them J13 685119136923, Q12 PJE138K, Q2 PJE138K, U43 NTS0102, U44 TPD4E05U06QDQARQ1, U45 TPD4E05U06QDQARQ1, U46 TPD4E05U06QDQARQ1

Commit message: v2.0 Schematic updates
Other:
- company: Argus-1 Cubesat -> Carnegie Mellon University
- title: Jetson Carrier Board -> Argus Carrierboard
Changed lines of the file:
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@@
 	(paper "A3")
 	(title_block
-		(title "Jetson Carrier Board")
-		(date "2024-07-05")
-		(rev "v1")
-		(company "Argus-1 Cubesat")
+		(title "Argus Carrierboard")
+		(date "2025-03-10")
+		(rev "v2.0")
+		(company "Carnegie Mellon University")
 		(comment 1 "www.antmicro.com")
 		(comment 2 "N. Khera")
@@
 	(label "HDMI_CLK_CONN_N"
 		(at 308.61 149.86 0)
-		(fields_autoplaced yes)
 		(effects
 			(font
@@
 	(label "HDMI_HPD_5V"
 		(at 307.34 226.06 180)
-		(fields_autoplaced yes)
 		(effects
 			(font
@@
 	(label "HDMI_D0_P"
 		(at 208.28 139.7 0)
-		(fields_autoplaced yes)
 		(effects
 			(font
@@
 	(label "HDMI_D0_CONN_P"
 		(at 297.18 66.04 0)
-		(fields_autoplaced yes)
 		(effects
 			(font
@@
 	(label "HDMI_D1_N"
 		(at 208.28 134.62 0)
-		(fields_autoplaced yes)
 		(effects
 			(font
@@
 	(label "HDMI_HPD_5V"
 		(at 297.18 82.55 0)
-		(fields_autoplaced yes)
 		(effects
 			(font
@@
 	(label "HDMI_D2_N"
 		(at 208.28 127 0)
-		(fields_autoplaced yes)
 		(effects
 			(font
@@
 	(label "5V_HDMI"
 		(at 270.51 157.48 0)
-		(fields_autoplaced yes)
 		(effects
 			(font
@@
 	(label "5V_HDMI"
 		(at 334.01 175.26 0)
-		(fields_autoplaced yes)
 		(effects
 			(font
@@
 	(label "HDMI_D2_CONN_N"
 		(at 308.61 127 0)
-		(fields_autoplaced yes)
 		(effects
 			(font
@@
 	(label "HDMI_D0_CONN_P"
 		(at 308.61 139.7 0)
-		(fields_autoplaced yes)
 		(effects
 			(font
@@
 	(label "HDMI_SCL_3V3"
 		(at 223.52 154.94 0)
-		(fields_autoplaced yes)
 		(effects
 			(font
@@
 	(label "HDMI_SDA_5V"
 		(at 297.18 85.09 0)
-		(fields_autoplaced yes)
 		(effects
 			(font
@@
 	(label "HDMI_SDA_3V3"
 		(at 223.52 157.48 0)
-		(fields_autoplaced yes)
 		(effects
 			(font
@@
 	(label "HDMI_CLK_N"
 		(at 208.28 149.86 0)
-		(fields_autoplaced yes)
 		(effects
 			(font
@@
 	(label "HDMI_SCL_5V"
 		(at 308.61 154.94 0)
-		(fields_autoplaced yes)
 		(effects
 			(font
@@
 	(label "5V_HDMI"
 		(at 292.1 173.99 180)
-		(fields_autoplaced yes)
 		(effects
 			(font
@@
 	(label "HDMI_SCL_5V"
 		(at 297.18 87.63 0)
-		(fields_autoplaced yes)
 		(effects
 			(font
@@
 	(label "HDMI_CLK_CONN_P"
 		(at 308.61 147.32 0)
-		(fields_autoplaced yes)
 		(effects
 			(font
@@
 	(label "HDMI_D0_CONN_N"
 		(at 308.61 142.24 0)
-		(fields_autoplaced yes)
 		(effects
 			(font
@@
 	(label "HDMI_D0_CONN_N"
 		(at 297.18 63.5 0)
-		(fields_autoplaced yes)
 		(effects
 			(font
@@
 	(label "HDMI_HPD_5V_R"
 		(at 284.48 226.06 180)
-		(fields_autoplaced yes)
 		(effects
 			(font
@@
 	(label "HDMI_D1_P"
 		(at 208.28 132.08 0)
-		(fields_autoplaced yes)
 		(effects
 			(font
@@
 	(label "HDMI_CLK_P"
 		(at 208.28 147.32 0)
-		(fields_autoplaced yes)
 		(effects
 			(font
@@
 	(label "HDMI_D2_CONN_P"
 		(at 297.18 41.91 0)
-		(fields_autoplaced yes)
 		(effects
 			(font
@@
 	(label "HDMI_D1_CONN_N"
 		(at 297.18 34.29 0)
-		(fields_autoplaced yes)
 		(effects
 			(font
@@
 	(label "HDMI_D2_CONN_P"
 		(at 308.61 124.46 0)
-		(fields_autoplaced yes)
 		(effects
 			(font
@@
 	(label "HDMI_SDA_5V"
 		(at 308.61 157.48 0)
-		(fields_autoplaced yes)
 		(effects
 			(font
@@
 	(label "HDMI_CEC_5V"
 		(at 335.28 162.56 0)
-		(fields_autoplaced yes)
 		(effects
 			(font
@@
 	(label "HDMI_D1_CONN_P"
 		(at 308.61 132.08 0)
-		(fields_autoplaced yes)
 		(effects
 			(font
@@
 	(label "HDMI_CLK_CONN_P"
 		(at 297.18 60.96 0)
-		(fields_autoplaced yes)
 		(effects
 			(font
@@
 	(label "HDMI_D1_CONN_N"
 		(at 308.61 134.62 0)
-		(fields_autoplaced yes)
 		(effects
 			(font
@@
 	(label "HDMI_CLK_CONN_N"
 		(at 297.18 58.42 0)
-		(fields_autoplaced yes)
 		(effects
 			(font
@@
 	(label "HDMI_D2_P"
 		(at 208.28 124.46 0)
-		(fields_autoplaced yes)
 		(effects
 			(font
@@
 	(label "HDMI_D0_N"
 		(at 208.28 142.24 0)
-		(fields_autoplaced yes)
 		(effects
 			(font
@@
 	(label "HDMI_D2_CONN_N"
 		(at 297.18 39.37 0)
-		(fields_autoplaced yes)
 		(effects
 			(font
@@
 	(label "HDMI_HPD_5V"
 		(at 335.28 167.64 0)
-		(fields_autoplaced yes)
 		(effects
 			(font
@@
 	(label "HDMI_D1_CONN_P"
 		(at 297.18 36.83 0)
-		(fields_autoplaced yes)
 		(effects
 			(font
@@
 	(label "HDMI_CEC_5V"
 		(at 297.18 90.17 0)
-		(fields_autoplaced yes)
-		(effects
-			(font
+		(effects
+			(font

Commit message: v2.1 Updates
Parts:
- C45, C49, C50, C52, C86, C87, C88, C92: Author Antmicro -> (none); Dielectric X5R -> (none); License Apache-2.0 -> (none); MPN GRM155R61H104KE14D -> C85858; Val 100n -> (none); Voltage 50V -> (none)
- C51: Author Antmicro -> (none); License Apache-2.0 -> (none); MPN GRM188R61A106KE69D -> C697423; Manufacturer Murata -> (none); Val 10u -> (none)
- C98, C99: Author Antmicro -> (none); Dielectric X5R -> (none); License Apache-2.0 -> (none); MPN GRM155R61H104KE14D -> C307348; Val 100n -> (none); Voltage 50V -> (none)
- FB2: Author Antmicro -> (none); License Apache-2.0 -> (none); MPN BLM21PG221SN1D -> C85840; Manufacturer Murata -> (none)
- R132, R133, R134, R135, R136, R137, R138, R139: Author Antmicro -> (none); License Apache-2.0 -> (none); MPN CR0402-FX-4990GLF -> C2076754; Manufacturer Bourns -> (none); Public False -> (none); Tolerance 1% -> (none); Val 499R -> (none)
- R140, R141: Author Antmicro -> (none); Current 1A -> (none); License Apache-2.0 -> (none); MPN ERJ2GE0R00X -> C190119; Manufacturer Panasonic -> (none); Val 0R -> (none)
- R175, R176, R177, R179, TP22, TP5: now left out of the parts list
- R178, R49: Author Antmicro -> (none); License Apache-2.0 -> (none); MPN CR0402-FX-2201GLF -> C237792; Manufacturer Bourns -> (none); Tolerance 1% -> (none); Val 100k -> (none)
- R47: Author Antmicro -> (none); License Apache-2.0 -> (none); MPN CR0402-FX-1002GLF -> C2479067; Manufacturer Bourns -> (none); Tolerance 1% -> (none); Val 10k -> (none)
- U44, U45, U46: Author Antmicro -> (none); License Apache-2.0 -> (none); MPN TPD4E05U06QDQARQ1 -> C81353
Other:
- moved on the sheet: C99
