File: hdmi.kicad_sch (KiCad schematic)
At the start: 41 parts, among them J13 685119136923, Q12 PJE138K, Q2 PJE138K, U43 NTS0102, U44 TPD4E05U06QDQARQ1, U45 TPD4E05U06QDQARQ1, U46 TPD4E05U06QDQARQ1

Commit message: Finish HDMI routing, replace usbc w/ usba
Parts:
- U44, U45, U46: footprint JetsonCarrier:USON-10_2.5x1mm_P0.5mm -> Argus-Miscellaneous:USON-10_TEX

Commit message: Power routing, CSI length matching, cleanup
Parts:
- U43: footprint JetsonCarrier:XSON-8_1x1.95mm_P0.5mm -> Argus-IC:NXP_XSON-8
Changed lines of the file:
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@@
 			)
 		)
-		(property "Footprint" "JetsonCarrier:XSON-8_1x1.95mm_P0.5mm"
+		(property "Footprint" "Argus-IC:NXP_XSON-8"
 			(at 293.37 173.99 0)
 			(hide yes)

Commit message: Layout cleanup, silk
Parts:
- TP22, TP5: footprint JetsonCarrier:TP_SMD_0.75mm -> TestPoint:TestPoint_Pad_D1.0mm
Changed lines of the file:
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@@
 			)
 		)
-		(property "Footprint" "JetsonCarrier:TP_SMD_0.75mm"
+		(property "Footprint" "TestPoint:TestPoint_Pad_D1.0mm"
 			(at 237.49 215.9 0)
 			(hide yes)
@@
 			)
 		)
-		(property "Footprint" "JetsonCarrier:TP_SMD_0.75mm"
+		(property "Footprint" "TestPoint:TestPoint_Pad_D1.0mm"
 			(at 335.28 157.48 0)
 			(hide yes)

Commit message: route all diff pairs, length tuning
Parts:
- removed U43: NTS0102, Argus-IC:NXP_XSON-8, symbol JetsonCarrier:NTS0102
- added U12: NTS0102, Argus-IC:NXP_XSON-8, symbol Argus-IC:NTS0102
- renumbered C86 to C43, C87 to C44, C88 to C45, C92 to C46, C45 to C47, C49 to C48, C50 to C49, C52 to C50, C98 to C51, C99 to C52, C51 to C53, D20 to D14, J13 to J7, Q12 to Q3, R132 to R48, R133 to R49, R134 to R50, R135 to R51, R136 to R52, R137 to R53, R138 to R54, R139 to R55, R140 to R56, R141 to R57, R175 to R58, R176 to R59, R47 to R60, R177 to R61, R178 to R62, R179 to R63, R49 to R64, TP22 to TP8, TP5 to TP9, U44 to U13, U45 to U14, U46 to U15
Connections:
- net +3V3: now also U12.3 (VCC_{A}), U12.6 (OE)
- net 5V_HDMI: now also U12.7 (VCC_{B})
- net GND: now also U12.2 (GND)
- net HDMI_SCL_3V3: now also U12.4 (A_{2})
- net HDMI_SCL_5V: now also U12.1 (B_{2})
- net HDMI_SDA_3V3: now also U12.5 (A_{1})
- net HDMI_SDA_5V: now also U12.8 (B_{1})
