File: imu.kicad_sch (KiCad schematic)
At the start: 4 parts, among them U2 BMX160

Commit message: v2.1 Updates
Parts:
- C7, C8: value 0.1uF -> 100nF; MPN (none) -> C307348
- R16: MPN (none) -> C2479067
Other:
- company: (none) -> Carnegie Mellon University
- title: (none) -> Argus Carrierboard
Changed lines of the file:
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@@
 	(generator_version "9.0")
 	(paper "A4")
+	(title_block
+		(title "Argus Carrierboard")
+		(date "2025-06-17")
+		(rev "v2.1")
+		(company "Carnegie Mellon University")
+		(comment 1 "www.antmicro.com")
+		(comment 2 "N. Khera")
+	)
 	(text "0x68"
 		(exclude_from_sim no)
@@
 			)
 		)
+		(property "MPN" "C2479067"
+			(at 171.45 91.44 90)
+			(effects
+				(font
+					(size 1.27 1.27)
+				)
+				(hide yes)
+			)
+		)
 		(pin "1"
 		)
@@
 			)
 		)
-		(property "Value" "0.1uF"
+		(property "Value" "100nF"
 			(at 124.714 96.266 0)
 			(effects
@@
 		)
 		(property "Description" "Unpolarized capacitor, small symbol"
+			(at 127 95.25 0)
+			(effects
+				(font
+					(size 1.27 1.27)
+				)
+				(hide yes)
+			)
+		)
+		(property "MPN" "C307348"
 			(at 127 95.25 0)
 			(effects
@@
 			)
 		)
-		(property "Value" "0.1uF"
+		(property "Value" "100nF"
 			(at 173.482 105.664 0)
 			(effects
@@
 			(at 171.45 105.41 0)
 			(effects
+				(font
+					(size 1.27 1.27)
+				)
+				(hide yes)
+			)
+		)
+		(property "MPN" "C307348"
+			(at 171.45 105.41 0)
+			(effects
