File: imu.kicad_sch (KiCad schematic)
At the start: 4 parts, among them U2 BMX160

Commit message: Clean up silk, BOM
Parts:
- C7: LCSC (none) -> C84419
- C8: LCSC (none) -> C14663
- R16: LCSC (none) -> C17168
- U2: LCSC (none) -> C892821
Changed lines of the file:
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@@
+			)
+		)
+		(property "LCSC" "C17168"
+			(at 171.45 87.376 0)
+			(effects
+				(font
+					(size 1.27 1.27)
+				)
+				(hide yes)
 			)
 		)
@@
 			)
 		)
+		(property "LCSC" "C84419"
+			(at 124.968 94.488 0)
+			(effects
+				(font
+					(size 1.27 1.27)
+				)
+				(hide yes)
+			)
+		)
 		(pin "1"
 		)
@@
 			)
 		)
+		(property "LCSC" "C14663"
+			(at 173.482 103.886 0)
+			(effects
+				(font
+					(size 1.27 1.27)
+				)
+				(hide yes)
+			)
+		)
 		(pin "1"
 		)
@@
 			)
 		)
+		(property "LCSC" "C892821"
+			(at 149.86 87.63 0)
+			(effects
+				(font
+					(size 1.27 1.27)
+				)
+				(hide yes)
+			)
+		)
