File: m-2.kicad_sch (KiCad schematic)
At the start: 26 parts, among them J2 1-2199230-6, Y1 ECS-327MVATX-2-CN-TR3

Commit message: v2.0 Schematic updates
Other:
- company: Argus-1 Cubesat -> Carnegie Mellon University
- title: Jetson Carrier Board -> Argus Carrierboard
Changed lines of the file:
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@@
 	(paper "A3")
 	(title_block
-		(title "Jetson Carrier Board")
-		(date "2024-07-10")
-		(rev "v1")
-		(company "Argus-1 Cubesat")
+		(title "Argus Carrierboard")
+		(date "2025-03-10")
+		(rev "v2.0")
+		(company "Carnegie Mellon University")
 		(comment 1 "www.antmicro.com")
 		(comment 2 "N. Khera")
@@
 	(label "3V3_M2"
 		(at 246.38 92.71 0)
-		(fields_autoplaced yes)
 		(effects
 			(font
@@
 	(label "C_PCIE0_TX3_P"
 		(at 194.31 163.83 180)
-		(fields_autoplaced yes)
 		(effects
 			(font
@@
 	(label "C_PCIE0_TX2_N"
 		(at 195.58 151.13 180)
-		(fields_autoplaced yes)
 		(effects
 			(font
@@
 	(label "~{M2_M_ALERT}"
 		(at 229.87 123.19 0)
-		(fields_autoplaced yes)
 		(effects
 			(font
@@
 	(label "M2_M_SMB_DATA"
 		(at 229.87 125.73 0)
-		(fields_autoplaced yes)
 		(effects
 			(font
@@
 	(label "PCIE_WAKE_SEL0"
 		(at 91.44 107.95 180)
-		(fields_autoplaced yes)
 		(effects
 			(font
@@
 	(label "C_PCIE0_TX1_P"
 		(at 195.58 133.35 180)
-		(fields_autoplaced yes)
 		(effects
 			(font
@@
 	(label "M2_M_SMB_CLK"
 		(at 229.87 128.27 0)
-		(fields_autoplaced yes)
 		(effects
 			(font
@@
 	(label "C_PCIE0_TX2_P"
 		(at 195.58 148.59 180)
-		(fields_autoplaced yes)
 		(effects
 			(font
@@
 	(label "32.7KHZ_OUT"
 		(at 274.32 109.22 180)
-		(fields_autoplaced yes)
 		(effects
 			(font
@@
 	(label "C_PCIE0_TX0_N"
 		(at 195.58 120.65 180)
-		(fields_autoplaced yes)
 		(effects
 			(font
@@
 	(label "32.7KHZ_OUT"
 		(at 82.55 154.94 180)
-		(fields_autoplaced yes)
 		(effects
 			(font
@@
 	(label "M2_M_SUSCLK"
 		(at 243.84 109.22 180)
-		(fields_autoplaced yes)
 		(effects
 			(font
@@
 	(label "PCIE_WAKE_SEL0"
 		(at 158.75 101.6 0)
-		(fields_autoplaced yes)
 		(effects
 			(font
@@
 	(label "C_PCIE0_TX0_P"
 		(at 195.58 118.11 180)
-		(fields_autoplaced yes)
 		(effects
 			(font
@@
 	(label "C_PCIE0_TX1_N"
 		(at 195.58 135.89 180)
-		(fields_autoplaced yes)
 		(effects
 			(font
@@
 	(label "C_PCIE0_TX3_N"
 		(at 194.31 166.37 180)
-		(fields_autoplaced yes)
-		(effects
-			(font
+		(effects
+			(font

Commit message: v2.1 Updates
Parts:
- C13, C14, C15, C16, C17, C18, C20: Author Antmicro -> (none); License Apache-2.0 -> (none); MPN CC0402KRX5R6BB224 -> C126623; Manufacturer YAGEO -> (none); Public False -> (none); Val 220n -> (none)
- C19: Author Antmicro -> (none); License Apache-2.0 -> (none); MPN CC0402KRX5R6BB224 -> C126623; Manufacturer YAGEO -> (none); Public False -> (none); Val 220nF -> (none)
- C21, C23, C24: Author Antmicro -> (none); License Apache-2.0 -> (none); MPN GRM188R61A106KE69D -> C697423; Manufacturer Murata -> (none); Val 10u -> (none)
- C22: Author Antmicro -> (none); License Apache-2.0 -> (none); MPN GRM188R61A106KE69D -> C697423; Manufacturer Murata -> (none); Val 10uF -> (none)
- C25: Author Antmicro -> (none); Dielectric X5R -> (none); License Apache-2.0 -> (none); MPN GRM155R61H104KE14D -> C307348; Manufacturer Murata -> (none); Val 100n -> (none); Voltage 50V -> (none)
- D1: Author Antmicro -> (none); License Apache-2.0 -> (none); MPN LTST-C190GKT -> C2909774; Manufacturer Lite-On -> (none); Public False -> (none)
- H5: footprint JetsonCarrier:Spacer_Drill3.7mm_H2.5mm_9774025151R -> MountingHole:MountingHole_2.7mm_M2.5_DIN965_Pad_TopBottom
- J2: Author Antmicro -> (none); License Apache-2.0 -> (none); MPN 1-2199230-6 -> C4710843
- R13, R19: Author Antmicro -> (none); Current 1A -> (none); License Apache-2.0 -> (none); MPN ERJ2GE0R00X -> C190119; Manufacturer Panasonic -> (none); Val 0R -> (none)
- R143: Author Antmicro -> (none); License Apache-2.0 -> (none); MPN PMR03EZPJ000 -> C844915; Manufacturer ROHM Semiconductor -> (none); Max. Curr. 22.4A -> (none); Val 0R -> (none)
- R37, R38, TP10, TP11, TP12: now left out of the parts list
- R39: Author Antmicro -> (none); License Apache-2.0 -> (none); MPN (none) -> C844928; Manufacturer Bourns -> (none); Tolerance 1% -> (none); Val 3K3 -> (none)
