File: som.kicad_sch (KiCad schematic)
At the start: 36 parts, among them J15 Bus_DDR4_SODIMM_CUSTOM_Jetson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, U4 NTS0102

Commit message: v2.0 Schematic updates
Other:
- company: Argus-1 Cubesat -> Carnegie Mellon University
- title: Jetson Carrier Board -> Argus Carrierboard
Changed lines of the file:
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@@
 	(paper "A3")
 	(title_block
-		(title "Jetson Carrier Board")
-		(date "2024-07-05")
-		(rev "v1")
-		(company "Argus-1 Cubesat")
+		(title "Argus Carrierboard")
+		(date "2025-03-10")
+		(rev "v2.0")
+		(company "Carnegie Mellon University")
 		(comment 1 "www.antmicro.com")
 		(comment 2 "N. Khera")
@@
 	(label "~{FORCE_RECOVERY}"
 		(at 105.41 163.83 0)
-		(fields_autoplaced yes)
 		(effects
 			(font
@@
 	(label "DEBUG_TXD_1V8"
 		(at 45.72 257.81 0)
-		(fields_autoplaced yes)
 		(effects
 			(font
@@
 	(label "SoM_5V_IN"
 		(at 54.61 100.33 180)
-		(fields_autoplaced yes)
 		(effects
 			(font
@@
 	(label "PMIC_BBAT"
 		(at 53.34 142.24 180)
-		(fields_autoplaced yes)
 		(effects
 			(font
@@
 	(label "DEBUG_RXD_1V8"
 		(at 45.72 260.35 0)
-		(fields_autoplaced yes)
 		(effects
 			(font
@@
 	(label "DEBUG_RXD_1V8"
 		(at 215.9 67.31 180)
-		(fields_autoplaced yes)
 		(effects
 			(font
@@
 	(label "DEBUG_TXD_1V8"
 		(at 215.9 64.77 180)
-		(fields_autoplaced yes)
 		(effects
 			(font

Commit message: v2.0 Layout completed. Exported BOM and STEP files
Parts:
- removed TP4: TP_0.75mm_SMD, JetsonCarrier:TP_SMD_0.75mm, symbol Connector:TestPoint
Connections:
- net SPIO_MISO: no longer names the net of J15.93 (SPI0_MISO)
- net SPIO_MOSI: no longer names the net of J15.89 (SPI0_MOSI)
- net SPIO_SCK: no longer names the net of J15.91 (SPI0_SCK)
- net ~{SPI0_CS0}: no longer names the net of J15.95 (~{SPI0_CS0})
- no-connect marks 65 -> 70

Commit message: v2.1 Updates
Parts:
- BTN1: Author Antmicro -> (none); License Apache-2.0 -> (none); MPN KMR211NGLFS -> C221676; Manufacturer C&K -> (none)
- C1, C2, C3, C35, C36, C4, C46: Author Antmicro -> (none); License Apache-2.0 -> (none); MPN CL10A226MO7JZNC -> C2762594; Public False -> (none); Val 22u -> (none); Voltage 16V -> (none)
- C37, C38: Author Antmicro -> (none); Dielectric X5R -> (none); License Apache-2.0 -> (none); MPN GRM155R61H104KE14D -> C307348; Val 100n -> (none); Voltage 50V -> (none)
- D15: footprint Diode_SMD:D_SOD-882 -> Package_SON:Texas_DPY0002A_0.6x1mm_P0.65mm; Author Antmicro -> (none); License Apache-2.0 -> (none); MPN TPD1E0B04 -> C1975594; Manufacturer Texas Instruments -> (none)
- FB1: Author Antmicro -> (none); License Apache-2.0 -> (none); MPN 74279221100 -> C5355985; Manufacturer Würth Elektronik -> (none)
- H6, H7: footprint JetsonCarrier:Spacer_Drill3.7mm_H2.5mm_9774025151R -> MountingHole:MountingHole_2.7mm_M2.5_DIN965_Pad_TopBottom
- R11, R12, R4, R5, R84, R92, R93, R94, R95, R96, R97, R98: Author Antmicro -> (none); Current 1A -> (none); License Apache-2.0 -> (none); MPN ERJ2GE0R00X -> C190119; Manufacturer Panasonic -> (none); Val 0R -> (none)
- R174: Author Antmicro -> (none); License Apache-2.0 -> (none); MPN CR0402-FX-2201GLF -> C2076947; Manufacturer Bourns -> (none); Tolerance 1% -> (none); Val 2k2 -> (none)
- R31, R80: Author Antmicro -> (none); License Apache-2.0 -> (none); MPN CR0402-FX-4701GLF -> C482093; Manufacturer Bourns -> (none); Tolerance 1% -> (none); Val 200k -> (none)
- TP25, TP7: now left out of the parts list
Other:
- note added: "#TODO: USB PINS ARE PROBABLY WRONG"
- moved on the sheet: BT1, R174
