File: usb.kicad_sch (KiCad schematic)
At the start: 29 parts, among them J3 USB4105-GF-A, U11 TPD4E05U06QDQARQ1, U5 FT230X, U8 NCP730BMT330

Commit message: v2.0 Schematic updates
Other:
- company: Argus-1 Cubesat -> Carnegie Mellon University
- title: Jetson Carrier Board -> Argus Carrierboard
Changed lines of the file:
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@@
 	(paper "A3")
 	(title_block
-		(title "Jetson Carrier Board")
-		(date "2024-07-05")
-		(rev "v1")
-		(company "Argus-1 Cubesat")
+		(title "Argus Carrierboard")
+		(date "2025-03-10")
+		(rev "v2.0")
+		(company "Carnegie Mellon University")
 		(comment 1 "www.antmicro.com")
 		(comment 2 "N. Khera")
@@
 	(label "USB_FTDI_P"
 		(at 63.5 165.1 0)
-		(fields_autoplaced yes)
 		(effects
 			(font
@@
 	(label "FTDI_3V3"
 		(at 102.87 123.19 180)
-		(fields_autoplaced yes)
 		(effects
 			(font
@@
 	(label "USBC3_VBUS"
 		(at 281.94 133.35 0)
-		(fields_autoplaced yes)
 		(effects
 			(font
@@
 	(label "FTDI_LED_TX"
 		(at 114.3 173.99 0)
-		(fields_autoplaced yes)
 		(effects
 			(font
@@
 	(label "USB_FTDI_N"
 		(at 63.5 167.64 0)
-		(fields_autoplaced yes)
 		(effects
 			(font
@@
 	(label "USBC3_CC1"
 		(at 313.69 138.43 0)
-		(fields_autoplaced yes)
 		(effects
 			(font
@@
 	(label "USBC3_CC1"
 		(at 250.825 181.61 0)
-		(fields_autoplaced yes)
 		(effects
 			(font
@@
 	(label "USBC3_D_P"
 		(at 313.69 151.13 0)
-		(fields_autoplaced yes)
 		(effects
 			(font
@@
 	(label "USB_FTDI_P"
 		(at 281.94 151.13 0)
-		(fields_autoplaced yes)
 		(effects
 			(font
@@
 	(label "FTDI_CBUS3"
 		(at 125.73 176.53 180)
-		(fields_autoplaced yes)
 		(effects
 			(font
@@
 	(label "FTDI_CBUS0"
 		(at 125.73 168.91 180)
-		(fields_autoplaced yes)
 		(effects
 			(font
@@
 	(label "USBC3_CC2"
 		(at 313.69 140.97 0)
-		(fields_autoplaced yes)
 		(effects
 			(font
@@
 	(label "USBC3_D_N"
 		(at 250.825 186.69 0)
-		(fields_autoplaced yes)
 		(effects
 			(font
@@
 	(label "USBC3_CC2"
 		(at 250.825 189.23 0)
-		(fields_autoplaced yes)
 		(effects
 			(font
@@
 	(label "USBC3_D_N"
 		(at 313.69 148.59 0)
-		(fields_autoplaced yes)
 		(effects
 			(font
@@
 	(label "FTDI_3V3"
 		(at 50.165 171.45 0)
-		(fields_autoplaced yes)
 		(effects
 			(font
@@
 	(label "USBC3_VBUS"
 		(at 54.61 123.19 0)
-		(fields_autoplaced yes)
 		(effects
 			(font
@@
 	(label "USB_FTDI_N"
 		(at 281.94 148.59 0)
-		(fields_autoplaced yes)
 		(effects
 			(font
@@
 	(label "USBC3_D_P"
 		(at 250.825 184.15 0)
-		(fields_autoplaced yes)
 		(effects
 			(font
@@
 	(label "FTDI_LED_RX"
 		(at 114.3 171.45 0)
-		(fields_autoplaced yes)
-		(effects
-			(font
+		(effects
+			(font

Commit message: v2.1 Updates
Parts:
- C27, C29, C31: Author Antmicro -> (none); Dielectric X5R -> (none); License Apache-2.0 -> (none); MPN GRM155R61H104KE14D -> C307348; Val 100n -> (none); Voltage 50V -> (none)
- C32: Author Antmicro -> (none); License Apache-2.0 -> (none); MPN C1608X5R1E106M080AC -> C697423; Manufacturer TDK -> (none); Val 10u/25V -> (none)
- C34: Author Antmicro -> (none); License Apache-2.0 -> (none); MPN CC0402MRX5R5BB106 -> C697423; Manufacturer YAGEO -> (none); Public False -> (none); Val 10u -> (none)
- C42: Author Antmicro -> (none); License Apache-2.0 -> (none); MPN C0402C105M4PACTU -> C2214844; Manufacturer KEMET -> (none); Val 1u/16V -> (none)
- C64: Author Antmicro -> (none); Dielectric X5R -> (none); License Apache-2.0 -> (none); MPN GRM155R61H104KE14D -> C307348; Manufacturer Murata -> (none); Val 100n -> (none); Voltage 50V -> (none)
- C94, C95: Author Antmicro -> (none); Dielectric C0G -> (none); License Apache-2.0 -> (none); MPN C0402C470J5GACTU -> C126511; Manufacturer KEMET -> (none); Public False -> (none); Val 47p -> (none)
- D2, D3, D4: Author Antmicro -> (none); License Apache-2.0 -> (none); MPN LTST-C190GKT -> C2909774; Manufacturer Lite-On -> (none); Public False -> (none)
- D6: Author Antmicro -> (none); License Apache-2.0 -> (none); MPN DF2S30FS -> C87910; Manufacturer Toshiba -> (none)
- R100: Author Antmicro -> (none); License Apache-2.0 -> (none); MPN (none) -> C490833; Tolerance 1% -> (none)
- R105: Author Antmicro -> (none); License Apache-2.0 -> (none); MPN CR0402-FX-4701GLF -> C844931; Manufacturer Bourns -> (none); Tolerance 1% -> (none); Val 4k7 -> (none)
- R117: Author Antmicro -> (none); License Apache-2.0 -> (none); MPN CR0402-FX-27R0GLF -> C844545; Manufacturer Bourns -> (none); Tolerance 1% -> (none); Val 27R -> (none)
- R127: Author Antmicro -> (none); License Apache-2.0 -> (none); MPN CR0402-FX-27R0GLF -> C844545; Manufacturer Bourns -> (none); Tolerance 1% -> (none)
- R46: Author Antmicro -> (none); License Apache-2.0 -> (none); MPN CR0402-FX-1002GLF -> C2479067; Manufacturer Bourns -> (none); Tolerance 1% -> (none); Val 10k -> (none)
- R56, R57: Author Antmicro -> (none); Current 1A -> (none); License Apache-2.0 -> (none); MPN ERJ2GE0R00X -> C190119; Manufacturer Panasonic -> (none); Val 0R -> (none)
- R72, R73: Author Antmicro -> (none); License Apache-2.0 -> (none); MPN (none) -> C844928; Tolerance 1% -> (none); Val 3K3 -> (none)
- R99: Author Antmicro -> (none); License Apache-2.0 -> (none); MPN (none) -> C490833; Manufacturer Bourns -> (none); Tolerance 1% -> (none)
- TP15, TP16: now left out of the parts list
- U11: Author Antmicro -> (none); License Apache-2.0 -> (none); MPN TPD4E05U06QDQARQ1 -> C81353
- U5: Author Antmicro -> (none); License Apache-2.0 -> (none); MPN FT230XQ-R -> C128629; Manufacturer FTDI Chip -> (none)
- U8: Author Antmicro -> (none); License Apache-2.0 -> (none); MPN NCP730BMT330TBG -> C892821; Manufacturer ON Semiconductor -> (none)
