File: usb3.kicad_sch (KiCad schematic)
At the start: 50 parts, among them J5 632723300011, Q13 PJE138K, Q4 PJE138K, U17 HD3SS3220RNH, U18 AP22615A_TSOT26, U19 TPD4E05U06QDQARQ1, U20 TPD4E05U06QDQARQ1, U21 TPD4E05U06QDQARQ1

Commit message: v2.0 Schematic updates
Other:
- company: Argus-1 Cubesat -> Carnegie Mellon University
- title: Jetson Carrier Board -> Argus Carrierboard
Changed lines of the file:
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@@
 	(paper "A3")
 	(title_block
-		(title "Jetson Carrier Board")
-		(date "2024-07-05")
-		(rev "v1")
-		(company "Argus-1 Cubesat")
+		(title "Argus Carrierboard")
+		(date "2025-03-10")
+		(rev "v2.0")
+		(company "Carnegie Mellon University")
 		(comment 1 "www.antmicro.com")
 		(comment 2 "N. Khera")
@@
 	(label "USBC1_ISC_SCL"
 		(at 132.08 175.26 0)
-		(fields_autoplaced yes)
 		(effects
 			(font
@@
 	(label "USBC1_RX1_P"
 		(at 177.8 157.48 0)
-		(fields_autoplaced yes)
 		(effects
 			(font
@@
 	(label "USBC1_ISET"
 		(at 251.46 90.17 0)
-		(fields_autoplaced yes)
 		(effects
 			(font
@@
 	(label "USBC1_I2C_SDA"
 		(at 132.08 172.72 0)
-		(fields_autoplaced yes)
 		(effects
 			(font
@@
 	(label "USBC1_CONN_TX2_P"
 		(at 222.25 180.34 0)
-		(fields_autoplaced yes)
 		(effects
 			(font
@@
 	(label "USBC1_CONN_TX2_N"
 		(at 222.25 177.8 0)
-		(fields_autoplaced yes)
 		(effects
 			(font
@@
 	(label "USBC1_FAULT_N"
 		(at 177.8 124.46 0)
-		(fields_autoplaced yes)
 		(effects
 			(font
@@
 	(label "USBC1_CONN_TX1_N"
 		(at 222.25 162.56 0)
-		(fields_autoplaced yes)
 		(effects
 			(font
@@
 	(label "USBC1_INT"
 		(at 132.08 177.8 0)
-		(fields_autoplaced yes)
 		(effects
 			(font
@@
 	(label "USBC1_CONN_TX1_P"
 		(at 222.25 165.1 0)
-		(fields_autoplaced yes)
 		(effects
 			(font
@@
 	(label "USBC1_PORT"
 		(at 132.08 137.16 0)
-		(fields_autoplaced yes)
 		(effects
 			(font
@@
 	(label "USBC1_TX2_N"
 		(at 177.8 177.8 0)
-		(fields_autoplaced yes)
 		(effects
 			(font
@@
 	(label "USBSS1_C_RX_P"
 		(at 132.08 157.48 0)
-		(fields_autoplaced yes)
 		(effects
 			(font
@@
 	(label "USBC1_TX1_N"
 		(at 177.8 162.56 0)
-		(fields_autoplaced yes)
 		(effects
 			(font
@@
 	(label "USBSS1_C_TX_N"
 		(at 132.08 162.56 0)
-		(fields_autoplaced yes)
 		(effects
 			(font
@@
 	(label "USBC1_ISC_SCL"
 		(at 104.14 193.04 0)
-		(fields_autoplaced yes)
 		(effects
 			(font
@@
 	(label "~{USBC1_EN_MUX}"
 		(at 132.08 139.7 0)
-		(fields_autoplaced yes)
 		(effects
 			(font
@@
 	(label "USBC1_VBUS_DET"
 		(at 177.8 129.54 0)
-		(fields_autoplaced yes)
 		(effects
 			(font
@@
 	(label "USBC1_CC2"
 		(at 222.25 137.16 0)
-		(fields_autoplaced yes)
 		(effects
 			(font
@@
 	(label "USBC1_TX2_P"
 		(at 177.8 180.34 0)
-		(fields_autoplaced yes)
 		(effects
 			(font
@@
 	(label "USBC1_I_MODE"
 		(at 132.08 134.62 0)
-		(fields_autoplaced yes)
 		(effects
 			(font
@@
 	(label "USBC1_VBUS"
 		(at 251.46 87.63 0)
-		(fields_autoplaced yes)
 		(effects
 			(font
@@
 	(label "USBSS1_C_TX_P"
 		(at 132.08 165.1 0)
-		(fields_autoplaced yes)
 		(effects
 			(font
@@
 	(label "USBC1_TX1_P"
 		(at 177.8 165.1 0)
-		(fields_autoplaced yes)
 		(effects
 			(font
@@
 	(label "USBC1_ID"
 		(at 311.15 69.85 0)
-		(fields_autoplaced yes)
 		(effects
 			(font
@@
 	(label "USBC1_I2C_SDA"
 		(at 104.14 190.5 0)
-		(fields_autoplaced yes)
 		(effects
 			(font
@@
 	(label "USBSS1_C_RX_N"
 		(at 132.08 154.94 0)
-		(fields_autoplaced yes)
 		(effects
 			(font
@@
 	(label "USBC1_CC1"
 		(at 222.25 134.62 0)
-		(fields_autoplaced yes)
 		(effects
 			(font
@@
 	(label "~{USBC1_EN_CC}"
 		(at 132.08 142.24 0)
-		(fields_autoplaced yes)
 		(effects
 			(font
@@
 	(label "USBC1_ADDR"
 		(at 132.08 170.18 0)
-		(fields_autoplaced yes)
 		(effects
 			(font
@@
 	(label "USBC1_RX1_N"
 		(at 177.8 154.94 0)
-		(fields_autoplaced yes)
 		(effects
 			(font
@@
 	(label "USBC1_ID"
 		(at 177.8 121.92 0)
-		(fields_autoplaced yes)
 		(effects
 			(font
@@
 	(label "USBC1_RX2_N"
 		(at 177.8 170.18 0)
-		(fields_autoplaced yes)
 		(effects
 			(font
@@
 	(label "USBC1_DIR"
 		(at 177.8 119.38 0)
-		(fields_autoplaced yes)
 		(effects
 			(font
@@
 	(label "USBC1_RX2_P"
 		(at 177.8 172.72 0)
-		(fields_autoplaced yes)
-		(effects
-			(font
+		(effects
+			(font

Commit message: v2.1 Updates
Parts:
- C67, C68, C69, C70, C71, C72: Author Antmicro -> (none); Dielectric X5R -> (none); License Apache-2.0 -> (none); MPN GRM155R61H104KE14D -> C85858; Manufacturer Murata -> (none); Val 100n -> (none); Voltage 50V -> (none)
- C73, C75: Author Antmicro -> (none); Dielectric X5R -> (none); License Apache-2.0 -> (none); MPN GRM155R61H104KE14D -> C307348; Val 100n -> (none); Voltage 50V -> (none)
- C74: Author Antmicro -> (none); License Apache-2.0 -> (none); MPN GRM188R61A106KE69D -> C697423; Manufacturer Murata -> (none); Val 10u -> (none)
- D5: Author Antmicro -> (none); License Apache-2.0 -> (none); MPN ESD9X5.0ST5G -> C87910; Manufacturer ON Semiconductor -> (none)
- D9: Author Antmicro -> (none); License Apache-2.0 -> (none); MPN LTST-C190GKT -> C2909774; Manufacturer Lite-On -> (none); Public False -> (none)
- J5: Author Antmicro -> (none); License Apache-2.0 -> (none); MPN 632723300011 -> C2830802
- R103, R107, R108, R109, R118, R119: Author Antmicro -> (none); Current 1A -> (none); License Apache-2.0 -> (none); MPN ERJ2GE0R00X -> C190119; Manufacturer Panasonic -> (none); Val 0R -> (none)
- R110, R113, R114, R115, R124, R125, R23, R60, TP26, TP27: now left out of the parts list
- R111, R112: Author Antmicro -> (none); License Apache-2.0 -> (none); MPN CR0402-FX-2003GLF -> C482193; Manufacturer Bourns -> (none); Tolerance 1% -> (none); Val 4k7 -> (none)
- R116, R120, R122, R123, R129: Author Antmicro -> (none); License Apache-2.0 -> (none); MPN CR0402-FX-1002GLF -> C71617; Manufacturer Bourns -> (none); Tolerance 1% -> (none); Val 10k -> (none)
- R121: Author Antmicro -> (none); License Apache-2.0 -> (none); MPN CR0402-FX-1001GLF -> C71623; Manufacturer Bourns -> (none); Tolerance 1% -> (none); Val 1k -> (none)
- R126: Author Antmicro -> (none); License Apache-2.0 -> (none); MPN CR0402-FX-2003GLF -> C482093; Manufacturer Bourns -> (none); Tolerance 1% -> (none); Val 200k -> (none)
- R128: Author Antmicro -> (none); License Apache-2.0 -> (none); MPN ERJ-2RKF8873X -> C409935; Manufacturer Panasonic -> (none); Public False -> (none); Tolerance 1% -> (none); Val 887k -> (none)
- R130: Author Antmicro -> (none); License Apache-2.0 -> (none); MPN CR0402-FX-2201GLF -> C2076947; Manufacturer Bourns -> (none); Tolerance 1% -> (none); Val 2k2 -> (none)
- R131: Author Antmicro -> (none); License Apache-2.0 -> (none); MPN CR0402-FX-4700GLF -> C482193; Manufacturer Bourns -> (none); Tolerance 1% -> (none); Val 4k7 -> (none)
- R24: Author Antmicro -> (none); License Apache-2.0 -> (none); MPN CR0402-FX-1002GLF -> C2479067; Manufacturer Bourns -> (none); Tolerance 1% -> (none); Val 10k -> (none)
- R61: Author Antmicro -> (none); License Apache-2.0 -> (none); MPN CR0402-FX-2003GLF -> C118142; Manufacturer Bourns -> (none); Tolerance 1% -> (none); Val 200k -> (none)
- U17: Author Antmicro -> (none); License Apache-2.0 -> (none); MPN HD3SS3220RNHT -> C165155
- U18: value AP22615A_TSOT26 -> AP22615A; Author Antmicro -> (none); License Apache-2.0 -> (none); MPN AP22615AWU-7 -> C2680357; Manufacturer Diodes Incorporated -> (none)
- U19, U20, U21: Author Antmicro -> (none); License Apache-2.0 -> (none); MPN TPD4E05U06QDQARQ1 -> C81353
Other:
- moved on the sheet: R115, R116, R118, R119
