File: supply.kicad_sch (KiCad schematic)
At the start: 110 parts, among them J11 282834-4, Q1 BSS138DWQ-7, Q10 MBT2222ADW1T1, Q11 PJE138K, Q5 PJE138K, Q6 SSM3J332R, Q7 MBT2222ADW1T1, Q8 PJE138K, Q9 BSS138DWQ-7, SW1 PCM12SMTR, U1 TPS56C230, U29 TPS56C230, U37 74LVC2G14, U38 74LVC1G175, U41 NCP730BMT330, U42 TPS7A0518P, U6 ADM1176-1ARMZ-R7

Commit message: v2.0 Schematic updates
Parts:
- removed BTN2: KMR211NGLFS, Button_Switch_SMD:SW_Push_1P1T-SH_NO_CK_KMR2xxG, symbol JetsonCarrier:SW_KMR211NGLFS_SMD
- removed D19: TPD1E0B04, Diode_SMD:D_SOD-882, symbol Device:D_TVS_Small
- added R147: 0R, Resistor_SMD:R_0603_1608Metric, symbol Device:R_Small
- R149: value 10k -> 0R; Author Antmicro -> (none); License Apache-2.0 -> (none); MPN CR0402-FX-1001GLF -> (none); Manufacturer Bourns -> (none); Tolerance 1% -> (none); Val 10k -> (none); now not fitted
Connections:
- net 3V3_STDB: now also R150.1; no longer R149.1
- net JETSON_EN: now also R149.1; no longer C53.1, D22.2 (A), R151.1, U37.1
- net VCC: now also SW1.1, R147.1; no longer U41.4 (EN)
- net A1: now reaches R91.1, U6.9 (A1)
- net at R149.2, SW1.2: now also U41.4 (EN), R147.2; no longer R150.1
- net A0: now reaches R62.1, U6.8 (A0)
- new net: C53.1, D22.2 (A), R151.1, U37.1
- no-connect marks 4 -> 3
Other:
- note added: "0x45"
- note added: "I2C1 ADDR"
- note added: "NOTE: SW1 STARTUP CRTL 1-2 AUTO 3-2 MAINBOARD"
- note removed: "NOTE: SW1 STARTUP CRTL 1-2 AUTO 3-2 MANUAL"
- note removed: "POWER BUTTON"
- note removed: "SHORT PRESS - POWER UP LONG PRESS - POWER DOWN"
- company: Argus-1 Cubesat -> Carnegie Mellon University
- title: Jetson Carrier Board -> Argus Carrierboard
- moved on the sheet: BTN3, C103, C105, C106, C107, C53, C54, C55, C56, C83, D16, D22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

Commit message: v2.0 Layout completed. Exported BOM and STEP files
Parts:
- removed C53, C54: 10uF, Capacitor_SMD:C_0603_1608Metric, symbol Device:C_Small
- removed C55, C56: 100nF, Capacitor_SMD:C_0603_1608Metric, symbol Device:C_Small
- removed D22, D23: RB521S30T1G, Diode_SMD:D_SOD-523, symbol Device:D_Schottky
- removed D24: VTVS8V5ASMF, Diode_SMD:D_SMF, symbol Device:D_Zener_Filled
- removed Q11: PJE138K, Package_TO_SOT_SMD:SOT-523, symbol JetsonCarrier:PJE138K
- removed R147, R149: 0R, Resistor_SMD:R_0603_1608Metric, symbol Device:R_Small
- removed R150, R151: 200k, Resistor_SMD:R_0603_1608Metric, symbol Device:R_Small
- removed R152: 200R, Resistor_SMD:R_0603_1608Metric, symbol Device:R_Small
- removed R154: 10k, Resistor_SMD:R_0603_1608Metric, symbol Device:R_Small
- removed U37: 74LVC2G14, Package_TO_SOT_SMD:SOT-23-6, symbol JetsonCarrier:74LVC2G14
- removed U38: 74LVC1G175, Package_TO_SOT_SMD:SOT-23-6, symbol JetsonCarrier:74LVC1G175
- added D7: 10V, Diode_SMD:D_SMA, symbol Device:D_Zener_Small
- added R14: 10k, Resistor_SMD:R_0603_1608Metric, symbol Device:R_Small
- SW1: value PCM12SMTR -> SW_SPDT; footprint Button_Switch_SMD:SW_SPDT_PCM12 -> JetsonCarrier:SW_SPDT_PCM12
Connections:
- net MB_3V3 is gone; now on net +3V3: R65.1, R68.1, R69.1, R76.1, R77.1, R78.1
- net 3V3_STDB: now also R14.2
- net GND: now also D7.2 (A)
- net JETSON_EN: now also SW1.1; no longer SW1.3
- net VBATT: now also D7.1 (K)
- net VCC: now also U41.4 (EN); no longer SW1.1
- net at SW1.2: now also R155.1; no longer U41.4 (EN)
- new net: R14.1, SW1.3
Other:
- note removed: "MODIFIED CIRCUIT FROM TI's SCEA048B AN"
- note removed: "NOTE: SW1 STARTUP CRTL 1-2 AUTO 3-2 MAINBOARD"
- moved on the sheet: C105, C106, D27, R155, R170, R181, TP23, U41

Commit message: v2.1 Updates
Parts:
- removed J11: 282834-4, JetsonCarrier:TE_282834-4, symbol Connector_Generic:Conn_01x04
- added J11: 205338-0002, JetsonCarrier:MOLEX_2053380002, symbol Connector_Generic_MountingPin:Conn_01x02_MountingPin
- added J4: 282834-2, JetsonCarrier:TE_282834-2, symbol Connector_Generic:Conn_01x02
- BTN3: Author Antmicro -> (none); License Apache-2.0 -> (none); MPN KMR211NGLFS -> C221676; Manufacturer C&K -> (none)
- C102, C103, C104, C6, C76: Author Antmicro -> (none); Dielectric X5R -> (none); License Apache-2.0 -> (none); MPN GRM155R61H104KE14D -> C307348; Val 100n -> (none); Voltage 50V -> (none)
- C105: Author Antmicro -> (none); License Apache-2.0 -> (none); MPN C1608X5R1E106M080AC -> C697423; Manufacturer TDK -> (none); Val 10u/25V -> (none)
- C106, C83: Author Antmicro -> (none); License Apache-2.0 -> (none); MPN CC0402MRX5R5BB106 -> C697423; Manufacturer YAGEO -> (none); Public False -> (none); Val 10u -> (none)
- C107, C93: Author Antmicro -> (none); License Apache-2.0 -> (none); MPN C1005X6S1A105K050BC -> C2214844; Manufacturer TDK -> (none); Val 1u -> (none)
- C26: MPN (none) -> C3877267; Val 3.3n -> (none)
- C28, C30: MPN (none) -> C161232; Val 10n -> (none)
- C77: Author Antmicro -> (none); License Apache-2.0 -> (none); MPN C1005X6S1A105K050BC -> C2214844; Manufacturer TDK -> (none); Val 1uF -> (none)
- C78, C80, C81, C82, C84, C85, C90, C91: Author Antmicro -> (none); License Apache-2.0 -> (none); MPN CL10A226MO7JZNC -> C2762594; Public False -> (none); Val 22u -> (none); Voltage 16V -> (none)
- D14: Author Antmicro -> (none); License Apache-2.0 -> (none); MPN LTST-C190GKT -> C2909774; Manufacturer Lite-On -> (none); Public False -> (none)
- D16: footprint Diode_SMD:D_SOD-882 -> Package_SON:Texas_DPY0002A_0.6x1mm_P0.65mm; Author Antmicro -> (none); License Apache-2.0 -> (none); MPN TPD1E0B04DPYR -> C1975594; Manufacturer Texas Instruments -> (none)
- D25: Author Antmicro -> (none); License Apache-2.0 -> (none); MPN ESD9X5.0ST5G -> C87910; Manufacturer ON Semiconductor -> (none)
- D26, D27: Author Antmicro -> (none); License Apache-2.0 -> (none); MPN ESD9X5.0ST5G -> C130456; Manufacturer ON Semiconductor -> (none)
- L1, L2: value XAL6030-182MEC -> XGL6030-182MEC
- Q1, Q9: Flight BSS138DWQ-7 -> (none); MPN (none) -> C3280240; Manufacturer_Name Diodes Incorporated -> (none); Manufacturer_Part_Number BSS138DWQ-7 -> (none); Proto BSS138DWQ-7 -> (none)
- R1: value ?R -> 10m; MPN (none) -> C840621
- R14: Author Antmicro -> (none); Current 1A -> (none); License Apache-2.0 -> (none); MPN ERJ2GE0R00X -> C2479067; Manufacturer Panasonic -> (none); Val 0R -> (none)
- R148, R157, R159, R161, R162, R172, R82: Author Antmicro -> (none); License Apache-2.0 -> (none); MPN CR0402-FX-1002GLF -> C2479067; Manufacturer Bourns -> (none); Tolerance 1% -> (none); Val 10k -> (none)
- R153: Author Antmicro -> (none); License Apache-2.0 -> (none); MPN CR0402-FX-2003GLF -> C118142; Manufacturer Bourns -> (none); Tolerance 1% -> (none); Val 200k -> (none)
- R155: footprint Resistor_SMD:R_0603_1608Metric -> Resistor_SMD:R_0402_1005Metric; Author Antmicro -> (none); Current 1A -> (none); License Apache-2.0 -> (none); MPN ERJ2GE0R00X -> C190119; Manufacturer Panasonic -> (none); Val 0R -> (none)
- R156, R158, R173, R181, TP21, TP23, TP24, TP28: now left out of the parts list
- R160, R167: Author Antmicro -> (none); Current 1A -> (none); License Apache-2.0 -> (none); MPN ERJ2GE0R00X -> C844915; Manufacturer Panasonic -> (none); Val 0R -> (none)
- R163: Author Antmicro -> (none); License Apache-2.0 -> (none); MPN CR0402-FX-1103GLF -> C473255; Manufacturer Bourns -> (none); Tolerance 1% -> (none); Val 110k -> (none)
- R164: Author Antmicro -> (none); License Apache-2.0 -> (none); MPN CR0402-FX-1502GLF -> C844742; Manufacturer Bourns -> (none); Tolerance 1% -> (none); Val 15k -> (none)
- R165: Author Antmicro -> (none); License Apache-2.0 -> (none); MPN CR0402-FX-9092GLF -> C403390; Manufacturer Bourns -> (none); Tolerance 1% -> (none); Val 90k9 -> (none)
- R166: Author Antmicro -> (none); License Apache-2.0 -> (none); MPN CR0402-FX-2002GLF -> C844923; Manufacturer Bourns -> (none); Tolerance 1% -> (none); Val 20k -> (none)
- R168, R169: Author Antmicro -> (none); License Apache-2.0 -> (none); MPN PMR03EZPJ000 -> C844934; Manufacturer ROHM Semiconductor -> (none); Max. Curr. 22.4A -> (none); Val 0R -> (none)
- R170, R171: Author Antmicro -> (none); Current 1A -> (none); License Apache-2.0 -> (none); MPN CR0603-J/-000ELF -> C844915; Manufacturer Bourns -> (none); Val 0R -> (none)
- R25: MPN (none) -> C2484712; Val 1k -> (none)
- R59, R75: MPN (none) -> C844802; Val 680R -> (none)
- R62: value 150k -> 0R; Val 150k -> 0R; now not fitted; now left out of the parts list
- R65, R76: MPN (none) -> C237792; Val 100k -> (none)
- R68, R69, R77, R78: MPN (none) -> C2479067; Val 10k -> (none)
- R70, R79: MPN (none) -> C118142; Val 200k -> (none)
- R71, R74: DNI DNI -> (none); DNP (none) -> DNP; now left out of the parts list
- R81: Author Antmicro -> (none); License Apache-2.0 -> (none); MPN CR0402-FX-2003GLF -> C2479067; Manufacturer Bourns -> (none); Tolerance 1% -> (none); Val 10k -> (none)
- R91: MPN (none) -> C402995; Val 150k -> (none)
- U1, U29: Author Antmicro -> (none); License Apache-2.0 -> (none); MPN TPS56C230RJER -> C1849534
- U41: Author Antmicro -> (none); License Apache-2.0 -> (none); MPN NCP730BMT330TBG -> C892821; Manufacturer ON Semiconductor -> (none)
- U42: Author Antmicro -> (none); License Apache-2.0 -> (none); MPN TPS7A0518PDBVT -> C2862322; Manufacturer Texas Instruments -> (none)
Connections:
- net +3V3: no longer R65.1, R68.1, R69.1, R76.1, R77.1, R78.1
- net 3V3_STDB: now also R65.1, R68.1, R69.1, R76.1, R77.1, R78.1
- net GND: now also J11.1 (Pin_1), J11.MP (MountPin), J4.1 (Pin_1)
- net VBATT: now also J11.2 (Pin_2), J4.2 (Pin_2)
Other:
- note added: "I2C ADDR 0x46"
- note added: "Rsense"
- note removed: "0x45"
- note removed: "I2C1 ADDR"
- moved on the sheet: D14, D7, R148

Commit message: Local Stash
Other:
- note added: "TODO: USE 3V3_STDB instead?"
Changed lines of the file:
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@@
+		)
+	)
+	(text "TODO: USE 3V3_STDB instead?"
+		(exclude_from_sim no)
+		(at 147.32 254.508 0)
+		(effects
+			(font
+				(size 2.54 2.54)
+			)
 		)
 	)
