File: jetson-orin-baseboard.kicad_pcb (KiCad board)
At the start: 8 copper layers, 90.2 x 95.9 mm, 406 parts, among them J1 522071560, J10 0533980471, J11 205338-0002, J12 522071560, J13 685119136923, J15 Bus_DDR4_SODIMM_CUSTOM_Jetson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, J2 1-2199230-6, J3 USB4105-GF-A, J4 282834-2, J5 632723300011, J6 522071560, J7 522711069, J8 522711069, J9 522071560, Q1 BSS138DWQ-7, Q10 MBT2222ADW1T1, Q12 PJE138K, Q13 PJE138K, Q2 PJE138K, Q4 PJE138K, Q5 PJE138K, Q6 SSM3J332R, Q7 MBT2222ADW1T1, Q8 PJE138K, Q9 BSS138DWQ-7, SW1 SW_SPDT, U1 TPS56C230, U11 TPD4E05U06QDQARQ1, U17 HD3SS3220RNH, U18 AP22615A, U19 TPD4E05U06QDQARQ1, U2 BMX160, U20 TPD4E05U06QDQARQ1, U21 TPD4E05U06QDQARQ1, U24 AP22615A, U25 AP22615A, U26 PI4MSD5V9548AZDEX, U29 TPS56C230, U3 AP22615A, U31 NTS0102, U32 NTS0102, U33 NTS0102, U4 NTS0102, U41 NCP730BMT330, U42 TPS7A0518P, U43 NTS0102, U44 TPD4E05U06QDQARQ1, U45 TPD4E05U06QDQARQ1, U46 TPD4E05U06QDQARQ1, U5 FT230X, U6 ADM1176-1ARMZ-R7, U7 AP22615A, U8 NCP730BMT330, U9 NTS0102, Y1 ECS-327MVATX-2-CN-TR3

Commit message: Initial layout attempt
Parts:
- removed C7, C8: 100nF, Capacitor_SMD:C_0603_1608Metric
- removed J1: 522071560, JetsonCarrier:CON_522071560_MOL
- removed J11: 205338-0002, JetsonCarrier:MOLEX_2053380002
- removed J4: 282834-2, JetsonCarrier:TE_282834-2
- removed R101, R102, R26, R55, R63: 2k2, Resistor_SMD:R_0402_1005Metric
- removed R16: 10k, Resistor_SMD:R_0603_1608Metric
- removed REF** (x2): , Calibration_Scale:Gauge_10mm_Type1_SilkScreenTop
- removed REF**: Val**, mainboard:XYZ_cubesat-top
- removed REF**: Val**, mainboard:XYZ_cubesat-bot
- removed U2: BMX160, JetsonCarrier:BMX160_BOS
- added H10: MountingHole_Pad, MountingHole:MountingHole_2.5mm_Pad_Via, F.Cu at (230.6, 95.5)
- added H9: MountingHole_Pad, MountingHole:MountingHole_2.5mm_Pad_Via, F.Cu at (230.6, 65.0)
- added J14: Conn_01x22_MountingPin, Connector_FFC-FPC:Amphenol_F32Q-1A7x1-11022_1x22-1MP_P0.5mm_Horizontal, B.Cu at (239.0, 80.2)
- added J16: Conn_01x22_MountingPin, Connector_FFC-FPC:Amphenol_F32Q-1A7x1-11022_1x22-1MP_P0.5mm_Horizontal, B.Cu at (154.8, 80.2)
- added J19: Conn_01x22_MountingPin, Connector_FFC-FPC:Amphenol_F32Q-1A7x1-11022_1x22-1MP_P0.5mm_Horizontal, B.Cu at (196.9, 38.1)
- added J20: Conn_01x22_MountingPin, Connector_FFC-FPC:Amphenol_F32Q-1A7x1-11022_1x22-1MP_P0.5mm_Horizontal, B.Cu at (196.9, 122.3)
- added J5: 632723300011, JetsonCarrier:USB-C_Receptacle_WE_632723300011, F.Cu at (278.4, 74.7)
- added R41: 2k2, Resistor_SMD:R_0402_1005Metric, F.Cu at (192.7, 39.0)
- added R42: 2k2, Resistor_SMD:R_0402_1005Metric, B.Cu at (202.2, 117.4)
- added R43: 2k2, Resistor_SMD:R_0402_1005Metric, F.Cu at (203.3, 124.8)
- added R52: 2k2, Resistor_SMD:R_0402_1005Metric, F.Cu at (192.5, 37.0)
- added R58: 2k2, Resistor_SMD:R_0402_1005Metric, F.Cu at (203.3, 128.8)
- C100, C101, C13, C14, C15, C16, C17, C18, C19, C20, C21, C22, C23, C24, C30, C96, C97, H5, H6, H7, J15, J2, R11, R12, R143, R155, R36, R4, R48, R5, R76, R77, R95, R96, R97, R98, SW1, U31, U32, kibuzzard-66A3478C: moved to F.Cu
- C25, C39, C43, C47, C79, R10, R13, R180, R182, R183, R184, R185, R19, R2, R3, R37, R38, R40, R50, R51, R6, R64, R66, R67, R7, R8, R85, R86, R9, TP10, TP11, TP12, TP21, U24, U25, U3, U7, Y1, kibuzzard-66A2E572, kibuzzard-66A2E636, kibuzzard-66A2E657: moved to B.Cu
- H1, H2, H3, H4: footprint JetsonCarrier:MountingHole2 -> MountingHole:MountingHole_3.2mm_M3_Pad_Via
- J12: value 522071560 -> QTH-030-01-L-D-A; footprint JetsonCarrier:CON_522071560_MOL -> Argus-Connectors:SAMTEC-QTH-030-01-X-D-A
- J6: value 522071560 -> 205338-0004; footprint JetsonCarrier:CON_522071560_MOL -> Connector_Molex:Molex_Pico-Lock_205338-0004_1x04-1MP_P2.00mm_Horizontal
- J8: value 522711069 -> 282834-4; footprint JetsonCarrier:CON_522711069_MOL -> Argus-Connectors:TE_282834-4
- J9: value 522071560 -> QSH-030-01-L-D-A; footprint JetsonCarrier:CON_522071560_MOL -> Argus-Connectors:SAMTEC_QSH-030-01-L-D-A; moved to B.Cu
- moved R90 219.9 mm to (319.8, 159.7)
- moved D13 219.9 mm to (316.8, 159.7)
- moved D10 200.0 mm to (334.8, 161.3)
- moved R87 200.0 mm to (334.8, 164.3)
- moved D12 167.3 mm to (303.3, 161.6)
- moved R89 167.3 mm to (303.3, 158.6)
- moved R76 162.9 mm to (334.1, 33.0), turned to 0 degrees
- moved H2 162.4 mm to (233.1, 37.4)
- moved R77 161.9 mm to (334.1, 31.2), turned to 0 degrees
- moved C30 161.5 mm to (334.7, 29.7), turned to 180 degrees
- moved Q1 161.2 mm to (326.2, 25.3)
- moved Q10 161.2 mm to (331.0, 21.3)
- moved Q7 161.2 mm to (326.2, 21.3)
- moved Q9 161.2 mm to (331.0, 25.3)
- moved R59 161.2 mm to (326.2, 19.3)
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Connections:
- J12 pad 1: /CSI/3V3_CAM3 -> VBATT
- J12 pad 10: CSI3_D1_P -> VBATT
- J12 pad 11: CSI3_D1_N -> GND
- J12 pad 13: CSI3_D0_P -> GND
- J12 pad 14: CSI3_D0_N -> GND
- J12 pad 2: /CSI/SDA_CAM3 -> VBATT
- J12 pad 3: /CSI/SCL_CAM3 -> VBATT
- J12 pad 4: MCLK_CAM3 -> VBATT
- J12 pad 5: /CSI/VSYNC_CAM3_3V3 -> VBATT
- J12 pad 6: GND -> VBATT
- J12 pad 7: CSI3_CLK_P -> VBATT
- J12 pad 8: CSI3_CLK_N -> VBATT
- J12 pad 9: GND -> VBATT
- J6 pad 1: /CSI/3V3_CAM1 -> VBATT
- J6 pad 2: /CSI/SDA_CAM1 -> VBATT
- J6 pad 3: /CSI/SCL_CAM1 -> GND
- J6 pad 4: MCLK_CAM1 -> GND
- J8 pad 1: GND -> VBATT
- J8 pad 2: /Peripherals/SHUTDOWN_REQ_MB -> VBATT
- J8 pad 3: MB_SDA -> GND
- J8 pad 4: MB_SCL -> GND
- J9 pad 1: /CSI/3V3_CAM2 -> VBATT
- J9 pad 10: CSI2_D1_P -> VBATT
- J9 pad 11: CSI2_D1_N -> GND
- J9 pad 13: CSI2_D0_P -> GND
- J9 pad 14: CSI2_D0_N -> GND
- J9 pad 2: /CSI/SDA_CAM2 -> VBATT
- J9 pad 3: /CSI/SCL_CAM2 -> VBATT
- J9 pad 4: MCLK_CAM2 -> VBATT
- J9 pad 5: /CSI/VSYNC_CAM2_3V3 -> VBATT
- J9 pad 6: GND -> VBATT
- J9 pad 7: CSI2_CLK_P -> VBATT
- J9 pad 8: CSI2_CLK_N -> VBATT
- J9 pad 9: GND -> VBATT
- R54 pad 2: /CSI/SCL_CAM0 -> /CSI/SCL_CAM2
Routing:
- net MB_SCL: track 172.0 -> 0.00 mm, vias 2 -> 0
- net MB_SDA: track 171.7 -> 0.00 mm, vias 2 -> 0
- net 3V3_STDB: track 187.2 -> 23.9 mm, vias 11 -> 0
- net ~{USBC1_INT}: track 138.4 -> 0.00 mm, vias 3 -> 0
- net GND: track 230.9 -> 106.7 mm, vias 386 -> 132
- net ~{RESET}: track 114.9 -> 2.68 mm, vias 5 -> 1
- net CSI3_D0_N: track 112.0 -> 0.00 mm, vias 2 -> 0
- net CSI3_D0_P: track 112.0 -> 0.00 mm, vias 2 -> 0
- net CSI3_D1_N: track 111.9 -> 0.00 mm, vias 2 -> 0
- net CSI3_CLK_N: track 111.9 -> 0.00 mm, vias 2 -> 0
- net CSI3_D1_P: track 111.9 -> 0.00 mm, vias 2 -> 0
- net CSI3_CLK_P: track 111.9 -> 0.00 mm, vias 2 -> 0
- net USBC1_PEN: track 105.5 -> 0.00 mm, vias 2 -> 0
- net SYS_SCL: track 104.9 -> 0.00 mm, vias 2 -> 0
- net CAM0_PEN: track 106.6 -> 3.36 mm, vias 3 -> 0
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- added copper zone on B.Cu, net (none)
- added copper zone on F.Cu, net (none)
- removed copper zone on F.Cu, net +1V8
- removed copper zone on In4.Cu, net +1V8
- removed copper zone on In4.Cu, net +3V3
- removed copper zone on F.Cu, net +5V
- removed copper zone on F.Cu, net /HDMI/5V_HDMI
- removed copper zone on B.Cu, net /M.2/3V3_M2
- removed copper zone on B.Cu, net /SoM/SoM_5V_IN
- removed copper zone on In4.Cu, net /USB Debug, USB2/FTDI_3V3
- removed copper zone on B.Cu, net /USB3, Recovery/USBC1_VBUS
- removed copper zone on B.Cu, net 5V_SoM
- removed copper zone on B.Cu, net GND
- removed copper zone on In6.Cu, net GND
- removed copper zone on In5.Cu, net Net-(Q2-D)
- removed copper zone on B.Cu, net VBATT
Other:
- board size 90.2 x 95.9 mm -> 189.2 x 105 mm
- board text added: "C20"
- board text added: "R168"
- board text removed: "15"
- board text removed: "CAM 3.3V"
- board text removed: "CAMERA 0"
- board text removed: "CAMERA 1"
- board text removed: "CAMERA 2"
- board text removed: "CAMERA 3"
- board text removed: "CLK+"
- board text removed: "CLK-"
- board text removed: "D0+"
- board text removed: "D0-"
- board text removed: "D1+"
- board text removed: "D1-"
- board text removed: "MCLK"
- board text removed: "TR"
- board text removed: "VSYNC"

Commit message: Finish HDMI routing, replace usbc w/ usba
Parts:
- removed C12: 1uF, Capacitor_SMD:C_0603_1608Metric
- removed C66: 10uF, Capacitor_SMD:C_0402_1005Metric
- removed C67, C68, C69, C70, C71, C72: 100nF, Capacitor_SMD:C_0402_1005Metric
- removed C73, C75: 100nF, Capacitor_SMD:C_0603_1608Metric
- removed C74: 10uF, Capacitor_SMD:C_0603_1608Metric
- removed D5: ESD9X5.0ST5G, Diode_SMD:D_SOD-923
- removed D9: LED_G_0603_LTST-C190GKT, LED_SMD:LED_0603_1608Metric
- removed J5 (x2): 632723300011, JetsonCarrier:USB-C_Receptacle_WE_632723300011
- removed J7: 522711069, JetsonCarrier:CON_522711069_MOL
- removed Q13, Q4: PJE138K, Package_TO_SOT_SMD:SOT-523
- removed R103, R107, R108, R109, R110, R113, R114, R118, R119, R124, R125: 0R, Resistor_SMD:R_0402_1005Metric
- removed R111, R112, R131: 4k7, Resistor_SMD:R_0402_1005Metric
- removed R115, R116, R120, R122, R123, R129: 10k, Resistor_SMD:R_0402_1005Metric
- removed R121: 1k, Resistor_SMD:R_0402_1005Metric
- removed R126: 200k, Resistor_SMD:R_0402_1005Metric
- removed R128: 887k, Resistor_SMD:R_0402_1005Metric
- removed R130: 2k2, Resistor_SMD:R_0402_1005Metric
- removed R23: 0R, Resistor_SMD:R_0603_1608Metric
- removed R24, R60: 10k, Resistor_SMD:R_0603_1608Metric
- removed R61: 200k, Resistor_SMD:R_0603_1608Metric
- removed TP26, TP27: TP_0.75mm_SMD, JetsonCarrier:TP_SMD_0.75mm
- removed U17: HD3SS3220RNH, JetsonCarrier:WQFN-30-1EP_4.6x2.6mm_P0.4mm
- removed U18: AP22615A, Package_TO_SOT_SMD:TSOT-23-6
- removed U19, U20, U21: TPD4E05U06QDQARQ1, JetsonCarrier:USON-10_2.5x1mm_P0.5mm
- added C108: 100nF, Capacitor_SMD:C_0603_1608Metric, B.Cu at (162.5, 94.8)
- added C110: 100nF, Capacitor_SMD:C_0402_1005Metric, B.Cu at (189.4, 70.6)
- added C111: 100nF, Capacitor_SMD:C_0402_1005Metric, B.Cu at (189.4, 69.6)
- added C112: 100nF, Capacitor_SMD:C_0603_1608Metric, B.Cu at (167.5, 71.6)
- added C113: 10uF, Capacitor_SMD:C_0603_1608Metric, B.Cu at (169.5, 68.0)
- added C114: 100nF, Capacitor_SMD:C_0603_1608Metric, B.Cu at (169.5, 66.4)
- added C115: 100nF, Capacitor_SMD:C_0402_1005Metric, B.Cu at (230.3, 104.0)
- added C116: 100nF, Capacitor_SMD:C_0402_1005Metric, B.Cu at (230.3, 105.0)
- added C117: 100nF, Capacitor_SMD:C_0603_1608Metric, F.Cu at (244.4, 97.1)
- added C118: 10uF, Capacitor_SMD:C_0603_1608Metric, F.Cu at (244.4, 99.6)
- added C119: 100nF, Capacitor_SMD:C_0603_1608Metric, F.Cu at (244.4, 102.1)
- added D17: ESD9X5.0ST5G, Diode_SMD:D_SOD-923, B.Cu at (162.2, 81.8)
- added D18: LED_G_0603_LTST-C190GKT, LED_SMD:LED_0603_1608Metric, B.Cu at (159.3, 52.5)
- added D19: LED_G_0603_LTST-C190GKT, LED_SMD:LED_0603_1608Metric, B.Cu at (155.5, 92.7)
- added D23: ESD9X5.0ST5G, Diode_SMD:D_SOD-923, F.Cu at (251.8, 106.5)
- added D24: LED_G_0603_LTST-C190GKT, LED_SMD:LED_0603_1608Metric, F.Cu at (248.4, 110.0)
- added D29: ESD9X5.0ST5G, Diode_SMD:D_SOD-923, B.Cu at (161.8, 95.9)
- added J1: USB3_A, Connector_USB:USB3_A_Molex_48393-001, B.Cu at (164.4, 64.7)
- added J17: Conn_01x15_MountingPin, Connector_FFC-FPC:Amphenol_F32Q-1A7x1-11015_1x15-1MP_P0.5mm_Horizontal, B.Cu at (239.0, 101.2)
- added J4: USB4105-GF-A, Connector_USB:USB_C_Receptacle_GCT_USB4105-xx-A_16P_TopMnt_Horizontal, B.Cu at (155.7, 99.2)
- added R101: 5k1, Resistor_SMD:R_0402_1005Metric, B.Cu at (161.9, 101.1)
- added R102: 5k1, Resistor_SMD:R_0402_1005Metric, B.Cu at (162.0, 96.9)
- added R106: 4k7, Resistor_SMD:R_0603_1608Metric, B.Cu at (158.5, 92.7)
- added R145: 0R, Resistor_SMD:R_0402_1005Metric, B.Cu at (230.3, 103.0)
- added R146: 0R, Resistor_SMD:R_0402_1005Metric, B.Cu at (230.3, 102.0)
- added R149: 1k, Resistor_SMD:R_0402_1005Metric, B.Cu at (173.7, 72.2)
- added R150: 1k, Resistor_SMD:R_0402_1005Metric, F.Cu at (262.4, 94.5)
- added R151: 10k, Resistor_SMD:R_0402_1005Metric, B.Cu at (173.7, 70.0)
- added R152: 10k, Resistor_SMD:R_0402_1005Metric, B.Cu at (172.5, 72.2)
- added R154: 2k2, Resistor_SMD:R_0402_1005Metric, B.Cu at (170.7, 73.8)
- added R186: 4k7, Resistor_SMD:R_0402_1005Metric, B.Cu at (159.3, 50.7)
- added R187: 10k, Resistor_SMD:R_0402_1005Metric, F.Cu at (265.3, 94.5)
- added R188: 10k, Resistor_SMD:R_0402_1005Metric, F.Cu at (265.3, 96.5)
- added R189: 2k2, Resistor_SMD:R_0402_1005Metric, F.Cu at (265.3, 98.5)
- added R190: 4k7, Resistor_SMD:R_0402_1005Metric, F.Cu at (265.3, 100.5)
- added U22: TPD4E05U06QDQARQ1, Argus-Miscellaneous:USON-10_TEX, B.Cu at (169.5, 59.0)
- added U23: TPD4E05U06QDQARQ1, Argus-Miscellaneous:USON-10_TEX, B.Cu at (169.5, 63.5)
- added U27: AP22615A, Package_TO_SOT_SMD:TSOT-23-6, B.Cu at (170.1, 71.0)
- added U28: TPD4E05U06QDQARQ1, Argus-Miscellaneous:USON-10_TEX, B.Cu at (162.0, 99.0)
- added U30: AP22615A, Package_TO_SOT_SMD:TSOT-23-6, F.Cu at (260.6, 110.5)
- added U34: TPD4E05U06QDQARQ1, Argus-Miscellaneous:USON-10_TEX, B.Cu at (233.3, 100.2)
- added U35: TPD4E05U06QDQARQ1, Argus-Miscellaneous:USON-10_TEX, B.Cu at (233.3, 103.5)
- C27, C29, C31, C32, C34, C42, C45, C49, C50, C52, C64, C86, C87, C88, C92, C94, C95, D2, D3, D4, D6, J13, J3, R100, R105, R117, R127, R132, R133, R134, R135, R136, R137, R138, R139, R140, R141, R175, R176, R46, R56, R57, R72, R73, R99, RN1, RN2, TP15, TP16, U43, U5, U8: moved to B.Cu
- Q2, R177, R179: moved to F.Cu
- U11, U44, U45, U46: footprint JetsonCarrier:USON-10_2.5x1mm_P0.5mm -> Argus-Miscellaneous:USON-10_TEX; moved to B.Cu
- moved C79 118.5 mm to (301.9, 108.2)
- moved R185 118.5 mm to (301.9, 111.2)
- moved R50 118.5 mm to (296.2, 108.6)
- moved R51 118.5 mm to (296.2, 107.2)
- moved R67 118.5 mm to (296.2, 110.1)
- moved R86 118.5 mm to (299.4, 106.0)
- moved U7 118.5 mm to (299.4, 108.8)
- moved C39 118.5 mm to (301.5, 99.6)
- moved C43 118.5 mm to (310.3, 99.6)
- moved C47 118.5 mm to (310.3, 108.2)
- moved R10 118.5 mm to (304.7, 107.2)
- moved R180 118.5 mm to (295.9, 100.1)
- moved R182 118.5 mm to (301.5, 102.6)
- moved R183 118.5 mm to (310.3, 111.2)
- moved R184 118.5 mm to (310.3, 102.6)
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Connections:
- net /USB Debug, USB2/FTDI_3V3 renamed /Debug/FTDI_3V3
- net /USB Debug, USB2/FTDI_CBUS0 renamed /Debug/FTDI_CBUS0
- net /USB Debug, USB2/FTDI_CBUS3 renamed /Debug/FTDI_CBUS3
- net /USB Debug, USB2/FTDI_LED_RX renamed /Debug/FTDI_LED_RX
- net /USB Debug, USB2/FTDI_LED_TX renamed /Debug/FTDI_LED_TX
- net /USB Debug, USB2/USBC3_CC1 renamed /Debug/USBC3_CC1
- net /USB Debug, USB2/USBC3_D_N renamed /Debug/USBC3_D_N
- net /USB Debug, USB2/USBC3_VBUS renamed /Debug/USBC3_VBUS
- net /USB Debug, USB2/USB_FTDI_N renamed /Debug/USB_FTDI_N
- net /USB Debug, USB2/USB_FTDI_P renamed /Debug/USB_FTDI_P
- C95 pad 2: /USB Debug, USB2/USBC3_D_P -> /Debug/USBC3_D_P
- J15 pad 39: unconnected-(J15D-USBSS1_RX_N-Pad39) -> USBSS1_RX_N
- J15 pad 41: unconnected-(J15D-USBSS1_RX_P-Pad41) -> USBSS1_RX_P
- J15 pad 45: unconnected-(J15D-USBSS1_TX_N-Pad45) -> USBSS1_TX_N
- J15 pad 47: unconnected-(J15D-USBSS1_TX_P-Pad47) -> USBSS1_TX_P
- J15 pad 51: USBSS2_RX_N -> unconnected-(J15D-USBSS2_RX_N-Pad51)
- J15 pad 53: USBSS2_RX_P -> unconnected-(J15D-USBSS2_RX_P-Pad53)
- J15 pad 57: USBSS2_TX_N -> unconnected-(J15D-USBSS2_TX_N-Pad57)
- J15 pad 59: USBSS2_TX_P -> unconnected-(J15D-USBSS2_TX_P-Pad59)
- J3 pad A6: /USB Debug, USB2/USBC3_D_P -> /Debug/USBC3_D_P
- J3 pad B5: /USB Debug, USB2/USBC3_CC2 -> /Debug/USBC3_CC2
- J3 pad B6: /USB Debug, USB2/USBC3_D_P -> /Debug/USBC3_D_P
- R100 pad 1: /USB Debug, USB2/USBC3_CC2 -> /Debug/USBC3_CC2
- R127 pad 1: /USB Debug, USB2/USBC3_D_P -> /Debug/USBC3_D_P
- U11 pad 2: /USB Debug, USB2/USBC3_D_P -> /Debug/USBC3_CC2
- U11 pad 5: /USB Debug, USB2/USBC3_CC2 -> /Debug/USBC3_D_P
- U11 pad 6: /USB Debug, USB2/USBC3_CC2 -> /Debug/USBC3_D_P
- U11 pad 9: /USB Debug, USB2/USBC3_D_P -> /Debug/USBC3_CC2
Routing:
- net DP1_TXD0_HDMI_TX2_P: track 0.00 -> 33.8 mm, vias 0 -> 2
- net DP1_TXD1_HDMI_TX1_P: track 0.00 -> 33.8 mm, vias 0 -> 2
- net DP1_TXD2_HDMI_TX0_P: track 0.00 -> 33.8 mm, vias 0 -> 2
- net DP1_TXD0_HDMI_TX2_N: track 0.00 -> 33.8 mm, vias 0 -> 2
- net DP1_HDMI_AUX_P: track 0.00 -> 33.8 mm, vias 0 -> 1
- net DP1_TXD1_HDMI_TX1_N: track 0.00 -> 33.8 mm, vias 0 -> 2
- net DP1_TXD2_HDMI_TX0_N: track 0.00 -> 33.8 mm, vias 0 -> 2
- net DP1_HDMI_AUX_N: track 0.00 -> 33.8 mm, vias 0 -> 1
- net DP1_TXD3_HDMI_TXC_P: track 2.74 -> 33.8 mm, vias 1 -> 2
- net DP1_TXD3_HDMI_TXC_N: track 2.74 -> 33.8 mm, vias 1 -> 2
- net (no net): track 0.00 -> 7.76 mm
- net +3V3: track 8.44 -> 15.9 mm
- net +1V8: track 8.07 -> 12.5 mm
- net /Debug/FTDI_CBUS3: track 4.40 -> 0.00 mm
- net Net-(J15H-GPIO12/PWM): track 0.00 -> 3.57 mm
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Other:
- board size 189.2 x 105 mm -> 90.2 x 95.9 mm
- board text added: "U44"
- board text removed: "Z"
