File: jetson-orin-baseboard.kicad_pcb (KiCad board)
At the start: 8 copper layers, 90.2 x 95.9 mm, 414 parts, among them J1 Bus_DDR4_SODIMM_CUSTOM_Jetson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, J10 Conn_01x22_MountingPin, J11 Conn_01x22_MountingPin, J12 0533980471, J13 QSH-030-01-L-D-A, J14 QTH-030-01-L-D-A, J15 282834-4, J16 205338-0004, J2 1-2199230-6, J3 USB_C_Receptacle_USB2.0_16P, J4 USB3_A, J5 Conn_01x15_MountingPin, J6 USB_C_Receptacle_USB2.0_16P, J7 685119136923, J8 Conn_01x22_MountingPin, J9 Conn_01x22_MountingPin, Q1 BSS138, Q10 MBT2222ADW1T1, Q2 PJE138K, Q3 PJE138K, Q4 PJE138K, Q5 PJE138K, Q6 SSM3J332R, Q7 NX3008NBKS, Q8 MBT2222ADW1T1, Q9 NX3008NBKS, SW1 SW_SPDT, U1 NTS0102, U10 TPD4E05U06QDQARQ1, U11 TPD4E05U06QDQARQ1, U12 NTS0102, U13 TPD4E05U06QDQARQ1, U14 TPD4E05U06QDQARQ1, U15 TPD4E05U06QDQARQ1, U16 PI4MSD5V9548AZDEX, U17 AP22615A, U18 AP22615A, U19 AP22615A, U2 NCP730BMT330, U20 AP22615A, U21 NTS0102, U22 NTS0102, U23 NTS0102, U24 NTS0102, U25 NTS0102, U26 MAX3051, U27 74LVC1G08, U28 SN74LV1T32DCKR, U29 ADM1176-1ARMZ-R7, U3 FT230X, U30 NTS0102, U31 74HCS74, U32 TPS56C230, U33 TPS56C230, U34 NCP730BMT330, U35 TPS7A0518P, U4 TPD4E05U06QDQARQ1, U5 AP22615A, U6 AP22615A, U7 TPD4E05U06QDQARQ1, U8 TPD4E05U06QDQARQ1, U9 TPD4E05U06QDQARQ1, Y1 ECS-327MVATX-2-CN-TR3

Commit message: general cleanup
Parts:
- moved TP18 0.80 mm to (196.9, 67.7)
- moved kibuzzard-6AA4D12B 0.80 mm to (191.9, 67.7)
- moved TP1 0.38 mm to (196.9, 57.9)
- moved kibuzzard-6AA4D4DE 0.32 mm to (192.7, 57.9)
Routing:
- net /CSI/3V3_CAM1: track 80.6 -> 78.3 mm
- net /USB3, Recovery/USB2_VBUS: track 46.4 -> 45.4 mm
- net /CSI/3V3_CAM3: track 42.7 -> 42.1 mm
- net /CSI/VSYNC_CAM0_3V3: track 65.5 -> 66.0 mm
- net VBATT: vias 44 -> 42
- net GND: vias 312 -> 329
