File: jetson-orin-baseboard.kicad_pcb (KiCad board)
At the start: 8 copper layers, 90.2 x 95.9 mm, 416 parts, among them J1 Bus_DDR4_SODIMM_CUSTOM_Jetson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, J10 Conn_01x22_MountingPin, J11 Conn_01x22_MountingPin, J12 0533980471, J13 QSH-030-01-L-D-A, J14 QTH-030-01-L-D-A, J15 282834-4, J16 205338-0004, J2 1-2199230-6, J3 USB_C_Receptacle_USB2.0_16P, J4 USB3_A, J5 Conn_01x15_MountingPin, J6 USB_C_Receptacle_USB2.0_16P, J7 685119136923, J8 Conn_01x22_MountingPin, J9 Conn_01x22_MountingPin, Q1 BSS138, Q10 MBT2222ADW1T1, Q2 PJE138K, Q3 PJE138K, Q4 PJE138K, Q5 PJE138K, Q6 SSM3J332R, Q7 NX3008NBKS, Q8 MBT2222ADW1T1, Q9 NX3008NBKS, SW1 SW_SPDT, U1 NTS0102, U10 TPD4E05U06QDQARQ1, U11 TPD4E05U06QDQARQ1, U12 NTS0102, U13 TPD4E05U06QDQARQ1, U14 TPD4E05U06QDQARQ1, U15 TPD4E05U06QDQARQ1, U16 PI4MSD5V9548AZDEX, U17 AP22615A, U18 AP22615A, U19 AP22615A, U2 NCP730BMT330, U20 AP22615A, U21 NTS0102, U22 NTS0102, U23 NTS0102, U24 NTS0102, U25 NTS0102, U26 MAX3051, U27 74LVC1G08, U28 SN74LV1T32DCKR, U29 INA226-Q1, U3 FT230X, U30 NTS0102, U31 74HCS74, U32 TPS56C230, U33 TPS56C230, U34 NCP730BMT330, U35 TPS7A0518P, U4 TPD4E05U06QDQARQ1, U5 AP22615A, U6 AP22615A, U7 TPD4E05U06QDQARQ1, U8 TPD4E05U06QDQARQ1, U9 TPD4E05U06QDQARQ1, Y1 ECS-327MVATX-2-CN-TR3

Commit message: Final cleanup, production files
Parts:
- removed REF** (x2): Gauge_10mm_Type1_SilkScreenTop, Calibration_Scale:Gauge_10mm_Type1_SilkScreenTop
- removed REF**: Val**, mainboard:XYZ_cubesat-top
- C102: value 100n -> 100nF
- D24: value ESD1V8WT -> ESD5Z2.5T1G
- FB2: footprint Inductor_SMD:L_0603_1608Metric -> Inductor_SMD:L_0805_2012Metric
- Q1: value BSS138 -> 2N7002
- Q2, Q3, Q4, Q5: value PJE138K -> 2N7002; footprint Package_TO_SOT_SMD:SOT-523 -> Package_TO_SOT_SMD:SOT-23
- moved Q3 3.32 mm to (205.0, 118.4), turned to 0 degrees
- moved Q5 0.85 mm to (208.6, 55.2)
- moved R134 0.69 mm to (206.0, 54.6), turned to -90 degrees
- moved D1 0.36 mm to (206.6, 45.7)
- moved FB2 0.25 mm to (205.1, 115.6)
- moved Q6 0.17 mm to (206.3, 58.3)
Routing:
- net GND: track 311.9 -> 331.0 mm
- net /HDMI/HDMI_HPD_5V_R: track 2.86 -> 7.71 mm
- net +5V: track 199.3 -> 196.8 mm
- net ~{RESET}: track 41.1 -> 40.3 mm
- net DP1_HPD: track 56.5 -> 56.0 mm
