File: jetson-orin-baseboard.kicad_sch (KiCad schematic)
At the start: 4 parts

Commit message: Initial layout attempt
Parts:
- H1, H2, H3, H4: footprint JetsonCarrier:MountingHole2 -> MountingHole:MountingHole_3.2mm_M3_Pad_Via; DNI DNI -> (none); MPN 9774065151R -> (none); Public False -> (none)
Other:
- removed sheet IMU

Commit message: Finish HDMI routing, replace usbc w/ usba
Other:
- sheet USB Debug, USB2 renamed Debug
Changed lines of the file:
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@@
 			(color 0 0 0 0)
 		)
-		(property "Sheetname" "USB Debug, USB2"
+		(property "Sheetname" "Debug"
 			(at 133.604 72.6309 0)
 			(show_name no)
