File: csi.kicad_sch (KiCad schematic)
At the start: 69 parts, among them J1 522071560, J12 522071560, J6 522071560, J9 522071560, U24 AP22615A, U25 AP22615A, U26 PI4MSD5V9548AZDEX, U3 AP22615A, U31 NTS0102, U32 NTS0102, U7 AP22615A

Commit message: Initial layout attempt
Parts:
- removed J1, J12, J6, J9: 522071560, JetsonCarrier:CON_522071560_MOL, symbol Connector_Generic_MountingPin:Conn_01x15_MountingPin
- removed R101, R102, R26, R55, R63: 2k2, Resistor_SMD:R_0402_1005Metric, symbol Device:R_Small
- added J14, J16, J19, J20: Conn_01x22_MountingPin, Connector_FFC-FPC:Amphenol_F32Q-1A7x1-11022_1x22-1MP_P0.5mm_Horizontal, symbol Connector_Generic_MountingPin:Conn_01x22_MountingPin
- added R41, R42, R43, R52, R58: 2k2, Resistor_SMD:R_0402_1005Metric, symbol Device:R_Small
Connections:
- net +3V3: now also R41.1, R42.1, R43.1, R52.1, R58.1
- net 3V3_CAM0: now also J19.1 (Pin_1)
- net 3V3_CAM1: now also J14.1 (Pin_1)
- net 3V3_CAM2: now also J20.1 (Pin_1)
- net 3V3_CAM3: now also J16.1 (Pin_1)
- net CSI0_CLK_N: now also J19.15 (Pin_15)
- net CSI0_CLK_P: now also J19.14 (Pin_14)
- net CSI0_D0_N: now also J19.21 (Pin_21)
- net CSI0_D0_P: now also J19.20 (Pin_20)
- net CSI0_D1_N: now also J19.18 (Pin_18)
- net CSI0_D1_P: now also J19.17 (Pin_17)
- net CSI1_CLK_N: now also J14.15 (Pin_15)
- net CSI1_CLK_P: now also J14.14 (Pin_14)
- net CSI1_D0_N: now also J14.21 (Pin_21)
- net CSI1_D0_P: now also J14.20 (Pin_20)
- net CSI1_D1_N: now also J14.18 (Pin_18)
- net CSI1_D1_P: now also J14.17 (Pin_17)
- net CSI2_CLK_N: now also J20.15 (Pin_15)
- net CSI2_CLK_P: now also J20.14 (Pin_14)
- net CSI2_D0_N: now also J20.21 (Pin_21)
- net CSI2_D0_P: now also J20.20 (Pin_20)
- net CSI2_D1_N: now also J20.18 (Pin_18)
- net CSI2_D1_P: now also J20.17 (Pin_17)
- net CSI3_CLK_N: now also J16.15 (Pin_15)
- net CSI3_CLK_P: now also J16.14 (Pin_14)
- net CSI3_D0_N: now also J16.21 (Pin_21)
- net CSI3_D0_P: now also J16.20 (Pin_20)
- net CSI3_D1_N: now also J16.18 (Pin_18)
- net CSI3_D1_P: now also J16.17 (Pin_17)
- net GND: now also J14.10 (Pin_10), J14.13 (Pin_13), J14.16 (Pin_16), J14.19 (Pin_19), J14.22 (Pin_22), J14.4 (Pin_4), J14.7 (Pin_7), J14.MP (MountPin), J16.10 (Pin_10), J16.13 (Pin_13), J16.16 (Pin_16), J16.19 (Pin_19), J16.22 (Pin_22), J16.4 (Pin_4), J16.7 (Pin_7), J16.MP (MountPin), J19.10 (Pin_10), J19.13 (Pin_13), J19.16 (Pin_16), J19.19 (Pin_19), J19.22 (Pin_22), J19.4 (Pin_4), J19.7 (Pin_7), J19.MP (MountPin), J20.10 (Pin_10), J20.13 (Pin_13), J20.16 (Pin_16), J20.19 (Pin_19), J20.22 (Pin_22), J20.4 (Pin_4), J20.7 (Pin_7), J20.MP (MountPin)
- net MCLK_CAM0: now also J19.5 (Pin_5)
- net MCLK_CAM1: now also J14.5 (Pin_5)
- net MCLK_CAM2: now also J20.5 (Pin_5)
- net MCLK_CAM3: now also J16.5 (Pin_5)
- net SCL_CAM0: now also J19.3 (Pin_3), R52.2; no longer R54.2
- net SCL_CAM1: now also J14.3 (Pin_3)
- net SCL_CAM2: now also R54.2, J20.3 (Pin_3)
- net SCL_CAM3: now also J16.3 (Pin_3), R58.2
- net SDA_CAM0: now also J19.2 (Pin_2), R41.2
- net SDA_CAM1: now also J14.2 (Pin_2)
- net SDA_CAM2: now also J20.2 (Pin_2), R42.2
- net SDA_CAM3: now also J16.2 (Pin_2), R43.2
- net VSYNC_CAM0_3V3: now also J19.6 (Pin_6)
- net VSYNC_CAM1_3V3: now also J14.6 (Pin_6)
- net VSYNC_CAM2_3V3: now also J20.6 (Pin_6)
- net VSYNC_CAM3_3V3: now also J16.6 (Pin_6)
- new net CSI0_D2_N: J19.12 (Pin_12)
- new net CSI0_D2_P: J19.11 (Pin_11)
- new net CSI0_D3_N: J19.9 (Pin_9)
- new net CSI0_D3_P: J19.8 (Pin_8)
- new net CSI1_D2_N: J14.12 (Pin_12)
- new net CSI1_D2_P: J14.11 (Pin_11)
- new net CSI1_D3_N: J14.9 (Pin_9)
- new net CSI1_D3_P: J14.8 (Pin_8)
- new net CSI2_D2_N: J20.12 (Pin_12)
- new net CSI2_D2_P: J20.11 (Pin_11)
- new net CSI2_D3_N: J20.9 (Pin_9)
- new net CSI2_D3_P: J20.8 (Pin_8)
- new net CSI3_D2_N: J16.12 (Pin_12)
- new net CSI3_D2_P: J16.11 (Pin_11)
- new net CSI3_D3_N: J16.9 (Pin_9)
- new net CSI3_D3_P: J16.8 (Pin_8)
Other:
- note added: "Additional CSI lanes are unused/unconnected"
- moved on the sheet: C100, C101, C39, C43, C47, C79, C89, C96, C97, D10, D11, D12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

Commit message: Power routing, CSI length matching, cleanup
Parts:
- U31, U32: footprint JetsonCarrier:XSON-8_1x1.95mm_P0.5mm -> Argus-IC:NXP_XSON-8
Changed lines of the file:
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@@
 			)
 		)
-		(property "Footprint" "JetsonCarrier:XSON-8_1x1.95mm_P0.5mm"
+		(property "Footprint" "Argus-IC:NXP_XSON-8"
 			(at 379.73 200.66 0)
 			(hide yes)
@@
 			)
 		)
-		(property "Footprint" "JetsonCarrier:XSON-8_1x1.95mm_P0.5mm"
+		(property "Footprint" "Argus-IC:NXP_XSON-8"
 			(at 379.73 232.41 0)
 			(hide yes)

Commit message: Layout cleanup, silk
Parts:
- TP13, TP14, TP17, TP18, TP19, TP20, TP8, TP9: footprint JetsonCarrier:TP_SMD_0.75mm -> TestPoint:TestPoint_Pad_D1.0mm
Changed lines of the file:
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@@
 			)
 		)
-		(property "Footprint" "JetsonCarrier:TP_SMD_0.75mm"
+		(property "Footprint" "TestPoint:TestPoint_Pad_D1.0mm"
 			(at 106.68 109.22 0)
 			(hide yes)
@@
 			)
 		)
-		(property "Footprint" "JetsonCarrier:TP_SMD_0.75mm"
+		(property "Footprint" "TestPoint:TestPoint_Pad_D1.0mm"
 			(at 106.68 93.98 0)
 			(hide yes)
@@
 			)
 		)
-		(property "Footprint" "JetsonCarrier:TP_SMD_0.75mm"
+		(property "Footprint" "TestPoint:TestPoint_Pad_D1.0mm"
 			(at 106.68 119.38 0)
 			(hide yes)
@@
 			)
 		)
-		(property "Footprint" "JetsonCarrier:TP_SMD_0.75mm"
+		(property "Footprint" "TestPoint:TestPoint_Pad_D1.0mm"
 			(at 106.68 96.52 0)
 			(hide yes)
@@
 			)
 		)
-		(property "Footprint" "JetsonCarrier:TP_SMD_0.75mm"
+		(property "Footprint" "TestPoint:TestPoint_Pad_D1.0mm"
 			(at 106.68 116.84 0)
 			(hide yes)
@@
 			)
 		)
-		(property "Footprint" "JetsonCarrier:TP_SMD_0.75mm"
+		(property "Footprint" "TestPoint:TestPoint_Pad_D1.0mm"
 			(at 106.68 111.76 0)
 			(hide yes)
@@
 			)
 		)
-		(property "Footprint" "JetsonCarrier:TP_SMD_0.75mm"
+		(property "Footprint" "TestPoint:TestPoint_Pad_D1.0mm"
 			(at 106.68 104.14 0)
 			(hide yes)
@@
 			)
 		)
-		(property "Footprint" "JetsonCarrier:TP_SMD_0.75mm"
+		(property "Footprint" "TestPoint:TestPoint_Pad_D1.0mm"
 			(at 106.68 101.6 0)
 			(hide yes)

Commit message: route all diff pairs, length tuning
Parts:
- removed U31, U32: NTS0102, Argus-IC:NXP_XSON-8, symbol JetsonCarrier:NTS0102
- added U21, U22: NTS0102, Argus-IC:NXP_XSON-8, symbol Argus-IC:NTS0102
- R100: renamed from R58; footprint Resistor_SMD:R_0402_1005Metric -> Resistor_SMD:R_0603_1608Metric
- R101: renamed from R43; footprint Resistor_SMD:R_0402_1005Metric -> Resistor_SMD:R_0603_1608Metric
- R82: renamed from R52; footprint Resistor_SMD:R_0402_1005Metric -> Resistor_SMD:R_0603_1608Metric
- R83: renamed from R41; footprint Resistor_SMD:R_0402_1005Metric -> Resistor_SMD:R_0603_1608Metric
- R90: renamed from R48; footprint Resistor_SMD:R_0402_1005Metric -> Resistor_SMD:R_0603_1608Metric
- R91: renamed from R36; footprint Resistor_SMD:R_0402_1005Metric -> Resistor_SMD:R_0603_1608Metric
- R98: renamed from R54; footprint Resistor_SMD:R_0402_1005Metric -> Resistor_SMD:R_0603_1608Metric
- R99: renamed from R42; footprint Resistor_SMD:R_0402_1005Metric -> Resistor_SMD:R_0603_1608Metric
- renumbered C89 to C54, C39 to C55, C43 to C56, C47 to C57, C79 to C58, C96 to C59, C97 to C60, C100 to C61, C101 to C62, D12 to D15, D13 to D16, D11 to D17, D10 to D18, J20 to J10, J16 to J11, J19 to J8, J14 to J9, R34 to R65, R35 to R66, R53 to R67, R142 to R68, R144 to R69, R180 to R70, R2 to R71, R40 to R72, R6 to R73, R66 to R74, R3 to R75, R7 to R76, R8 to R77, R182 to R78, R89 to R79, R184 to R80, R90 to R81, R9 to R84, R10 to R85, R50 to R86, R51 to R87, R64 to R88, R67 to R89, R85 to R92, R86 to R93, R183 to R94, R88 to R95, R185 to R96, R87 to R97, TP8 to TP10, TP9 to TP11, TP13 to TP12, TP14 to TP13, TP17 to TP14, TP18 to TP15, TP19 to TP16, TP20 to TP17, U26 to U16, U24 to U17, U25 to U18, U3 to U19, U7 to U20
Connections:
- net +1V8: now also U21.3 (VCC_{A}), U21.6 (OE), U22.3 (VCC_{A}), U22.6 (OE)
- net +3V3: now also U21.7 (VCC_{B}), U22.7 (VCC_{B})
- net GND: now also U21.2 (GND), U22.2 (GND)
- net VSYNC_CAM0: now also U21.4 (A_{2})
- net VSYNC_CAM0_3V3: now also U21.1 (B_{2})
- net VSYNC_CAM1: now also U21.5 (A_{1})
- net VSYNC_CAM1_3V3: now also U21.8 (B_{1})
- net VSYNC_CAM2: now also U22.4 (A_{2})
- net VSYNC_CAM2_3V3: now also U22.1 (B_{2})
- net VSYNC_CAM3: now also U22.5 (A_{1})
- net VSYNC_CAM3_3V3: now also U22.8 (B_{1})
