File: _restore_backup_2026-09-04T09-51-43-778/som.kicad_sch (KiCad schematic)
At the start: 33 parts, among them J15 Bus_DDR4_SODIMM_CUSTOM_Jetson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, U4 NTS0102

Commit message: Add CSI, USB, HDMI, PCIe
Parts:
- added H6, H7: 9774065151, MountingHole:MountingHole_2.7mm_M2.5_DIN965_Pad_TopBottom, symbol Mechanical:MountingHole_Pad
- J15: footprint Argus-Miscellaneous:Jetson_Module_TE_2309409-1 -> JetsonCarrier:TE_2309413
Connections:
- net DEBUG_RXD: now also U4.1 (B_{2}); no longer U4.8 (B_{1})
- net DEBUG_RXD_1V8: now also U4.4 (A_{2}); no longer U4.5 (A_{1})
- net DEBUG_TXD: now also U4.8 (B_{1}); no longer U4.1 (B_{2})
- net DEBUG_TXD_1V8: now also U4.5 (A_{1}); no longer U4.4 (A_{2})
- net GND: now also H6.1, H7.1
- net USBSS2_RX_N: now reaches J15.51 (USBSS2_RX_N)
- net USBSS2_RX_P: now reaches J15.53 (USBSS2_RX_P)
- net USBSS2_TX_N: now reaches J15.57 (USBSS2_TX_N)
- net USBSS2_TX_P: now reaches J15.59 (USBSS2_TX_P)
- net USBSS1_RX_N: no longer names the net of J15.39 (USBSS1_RX_N)
- net USBSS1_RX_P: no longer names the net of J15.41 (USBSS1_RX_P)
- net USBSS1_TX_N: no longer names the net of J15.45 (USBSS1_TX_N)
- net USBSS1_TX_P: no longer names the net of J15.47 (USBSS1_TX_P)
Other:
- note added: "#TODO: USB PINS ARE PROBABLY WRONG"
